File: connector.sch (KiCad schematic (older format))
At the start: 3 parts

Commit message: agrego mas conectores y paso a pcb (todo mal!)
agregue conectores RJ45 para el encadenamiento spi y busyflag, pero no
para pulse.. es lo voy a mandar aparte porque es individual por cada
driver.. al igual que switch, y vere si alguna cosa mas.. en el rj me
sobran aun 2 pines.. ya vere que mando..lastima que no puedo mandar
pulse por ahi.. porque al ser 1 por driver necesito ir directo desde el
controlador.. sino como?... pase a pcb para ver que onda nada mas y
obvio me faltan definir los footprints de casi todo.. pero al menos
paso...orcad ya estaria llorando y no podria hacer nada...como sea, esta
bueno...sigo
Parts:
- removed J?: Conn_01x04, Connector_Phoenix_MSTB:PhoenixContact_MSTBA_2,5_4-G-5,08_1x04_P5.08mm_Horizontal, symbol Connector_Generic:Conn_01x04
- added J2, J3: Conn_01x04, Connector_Phoenix_MSTB:PhoenixContact_MSTBA_2,5_4-G-5,08_1x04_P5.08mm_Horizontal, symbol Connector_Generic:Conn_01x04
- added J4, J5: RJ45, Connector_RJ:RJ45_Amphenol_54602-x08_Horizontal, symbol Connector:RJ45
- gave numbers to parts that had none: 2
Connections:
- net labels added: Busy, CLK, CS, MotorA1, MotorA2, MotorB1, MotorB2, Pulse, SDI, SDO, Switch
- wire segments 4 -> 27
- no-connect marks 0 -> 6
Other:
- moved on the sheet: D1

Commit message: armo huella step01 y asigno casi todas las huellas
ahi hice el landpattern del steo01, que es un parto, pero quedo bueno..
al tiempo que aprendi a editar y la verdad es que es comodo.. me animo a
decir que supera a allegro, y de hecho se parece demasiado en muchas
cosas.. huele a copia de algun lado.. incluiso los nombres en los menus
son iguales... como sea, ya quedo eso, lo que si tuve que volar algunos
pines repetidos en el simbolo porque sino era un chino tener muchos
pines repetidos, o sea en la huella tengo un pin que va a parar a
multiples pines en el esquemativo. si bien lo logre hacer superponiendo
encimados los pines en el esquemativo y dejandolos invisibles excepto
uno, eso funca, pero es un azco... preferi volar todos y dejar la union
univoca y listo.. al simbolo le faltan pines, pero el landpattern no los
necesita porque se unen todos en una misma masa de pad. despues pase
todas las huellas del resto del chiquitaje y ademas acomodo los power
netlist que estaban mal y de paso voy puliendo el disenio en general..
va quedando.. un poco mas y paso a tirar pista
Parts:
- added C7, C8: 100uFx100v, Capacitor_THT:CP_Radial_D12.5mm_P5.00mm, symbol Device:CP
- added J6: Conn_01x02, Connector_Phoenix_MSTB:PhoenixContact_MSTBA_2,5_2-G-5,08_1x02_P5.08mm_Horizontal, symbol Connector_Generic:Conn_01x02
- added JP1: jumper, Jumper:SolderJumper-2_P1.3mm_Open_RoundedPad1.0x1.5mm, symbol Jumper:SolderJumper_2_Open
Connections:
- net labels removed: 100V, 15V, 3V3, G15V
- wire segments 27 -> 35
- no-connect marks 6 -> 5
Other:
- note added: "Alimentacion"
- note added: "Cadena SPI con RJ45"
- note added: "Coneccion individual\n"
- note added: "Contemplo doble pin del conector para\npositivo y doble para negativo para \npermitir encadenar alimentacion y/o suplir\nmas corriente\n"
- note added: "Decido hacer el cruce de SPI en las fichas \ny no en el cable, de modo que los cables son\nsiempre rectos\n"
- note added: "El busy si se usa como salida para \nmanejar pulso a otro driver es individual"
- note added: "El fin de carrera y el step es individual \npor modulo asi que va por fuera \nde la cadena SPI\n"
- note added: "Potencia"
- note added: "segun las pruebas con 200uF \nsera suficiente para un ripple aceptable\n"
- note added: "si busy va de step, \nno va en cadena SPI, \nsino en conector individual\n"
- moved on the sheet: D1, J4, J5

Commit message: arranco a rutear, cambio xtal por SMD y opcion CLKIN
arranque a tirar pist porque me estaba aburriendo ya, de paso voy
practivcando los shortcuts y demas.. esta muy copado y te aviso.. es
plagio a allegro.. no cabe dudas.. como sea, cambie el Xtal por uno SMD
de 4 pines que se consigue y minimiza el espacio, agegue tambien clkin
para mandar clk a todos por igual con el PWM del uC para sincronizar con
un selector para poder usar el xtal si es que el PWM se pierde por
fanout o ruido.. y no mucho mas
Connections:
- net labels added: CLKIN
- wire segments 35 -> 37
- no-connect marks 5 -> 3
Changed lines of the file:
@@
 L Connector_Generic:Conn_01x04 J3
 U 1 1 5BC94397
-P 2050 5150
-F 0 "J3" H 1970 4725 50  0000 C CNN
-F 1 "Conn_01x04" H 1970 4816 50  0000 C CNN
-F 2 "Connector_Phoenix_MSTB:PhoenixContact_MSTBA_2,5_4-G-5,08_1x04_P5.08mm_Horizontal" H 2050 5150 50  0001 C CNN
-F 3 "~" H 2050 5150 50  0001 C CNN
-	1    2050 5150
-	-1   0    0    1
-$EndComp
+P 2050 5050
+F 0 "J3" H 1970 4625 50  0000 C CNN
+F 1 "Conn_01x04" H 1970 4716 50  0000 C CNN
+F 2 "Connector_Phoenix_MSTB:PhoenixContact_MSTBA_2,5_4-G-5,08_1x04_P5.08mm_Horizontal" H 2050 5050 50  0001 C CNN
+F 3 "~" H 2050 5050 50  0001 C CNN
+	1    2050 5050
+	-1   0    0    -1
+$EndComp
+Text HLabel 2400 4950 2    50   Input ~ 0
+MotorB2
+Text HLabel 2400 5250 2    50   Input ~ 0
+MotorA2
+Text HLabel 2400 5150 2    50   Input ~ 0
+MotorA1
 Text HLabel 2400 5050 2    50   Input ~ 0
-MotorB2
-Text HLabel 2400 5150 2    50   Input ~ 0
-MotorA2
-Text HLabel 2400 5250 2    50   Input ~ 0
-MotorA1
-Text HLabel 2400 4950 2    50   Input ~ 0
 MotorB1
 Wire Wire Line
@@
 	3700 2200 3700 2550
 NoConn ~ 7200 2250
-NoConn ~ 2550 2550
 NoConn ~ 2650 2550
-NoConn ~ 3800 2550
 NoConn ~ 3900 2550
 Text Notes 2300 3550 0    50   ~ 0
@@
 	0    1    1    0
 $EndComp
-Text Notes 2550 1450 0    50   ~ 0
+Text Notes 2700 1350 0    50   ~ 0
 si busy va de step, \nno va en cadena SPI, \nsino en conector individual\n
 Wire Wire Line
@@
 Text Notes 3800 6100 0    50   ~ 0
 Contemplo doble pin del conector para\npositivo y doble para negativo para \npermitir encadenar alimentacion y/o suplir\nmas corriente\n
+Text HLabel 3800 1700 1    50   Input ~ 0
+CLKIN
+Wire Wire Line
+	3800 1700 3800 2550
+Text HLabel 2550 1700 1    50   Input ~ 0
+CLKIN
+Wire Wire Line
+	2550 1700 2550 2550
 $EndSCHEMATC

Commit message: Cambio Rj's vuela xtal, entra Reset, agrego tornillos
Hago de todo un poco entre lo que saco el xtal porque ya probe que no se
necesita, elijo un IC que gnere 16Mhz y lo encadeno al resto, el RJ lo
cambie por otra que se parece mas a la que voy a usar, pero hay que
verificar, agregue un selector de osc, y agregue unos agujeros de
tornillos que no se si los quiero. va bien.. tengo que meterle mas al
ruteo
Parts:
- added JP301: Clk_Select, Jumper:SolderJumper-3_P2.0mm_Open_TrianglePad1.0x1.5mm, symbol Jumper:Jumper_3_Open
- added MH301, MH302: MountingHole, MountingHole:MountingHole_3.2mm_M3, symbol Mechanical:MountingHole
- J4, J5: footprint Connector_RJ:RJ45_Amphenol_54602-x08_Horizontal -> w_conn_pc:rj45-noshield
Connections:
- net labels added: Busy_Out, Osc, Osc_In, Osc_Out, Reset, Sdo_Chain
- net labels removed: CLKIN
- wire segments 37 -> 54
- no-connect marks 3 -> 1
Other:
- note added: "Holes"
- note added: "Main Power"
- note added: "Motor"
- note added: "Paralel Conn\n"
- note added: "Pins Selector"
- note added: "Spi Daisy Chain"
- note added: "si busy va de step, \nno va en cadena SPI, \nsino en conector \nindividual\n"
- note added: "un IC genera y el resto \nconsume CLK y regenera \ninvertido para el siguiente\nCon esto selecciono"
- note removed: "Alimentacion"
- note removed: "Cadena SPI con RJ45"
- note removed: "Coneccion individual\n"
- note removed: "Potencia"
- note removed: "si busy va de step, \nno va en cadena SPI, \nsino en conector individual\n"
- moved on the sheet: D1, J5

Commit message: cambio nombres, hago board edge, defino capas, posicion y demas
hice de todo un poco, principalmente le di forma a la placa con una
dimensino pasable, ajuste los conectores que aun no me convencen, pero
cambie la entrada para el conector de 4 y los motores en 2 de 2, cosa
que la alimentacion este toda en un solo conector y me queda piola para
que los motores salgan del IC para los costados. en cuanto a la logica
aun no me decido si voy a poner otra RJ para la salida d busy y demas o
meto bornera.. estouy mas del lado de la RJ y me quedaria genial para
poner los leds arriba de la RJ o a un costado.. puedo elegir eso.. mepa
que vamos con eso y asi no hay manera de mezclar fichas tampoco, porque
pongo un 6P6C RJ12 y ya.. hasta me sobran 2 pines.. bueno despues lo
sigo.
Parts:
- removed J4, J5: RJ45, w_conn_pc:rj45-noshield, symbol Connector:RJ45
- added rJ301: RJ45, pap:rj45_dci, symbol pap:RJ45
- added rJ302: RJ45, powerstep:rj45_dci, symbol pap:RJ45
- C7, C8: footprint Capacitor_THT:CP_Radial_D12.5mm_P5.00mm -> powerstep:CP_Radial_D13.0mm_P5.00mm
- J1, J6: footprint Connector_Phoenix_MSTB:PhoenixContact_MSTBA_2,5_2-G-5,08_1x02_P5.08mm_Horizontal -> powerstep:PhoenixContact_MSTBA_2,5_2-G-5,08_1x02_P5.08mm_Horizontal
- J2, J3: footprint Connector_Phoenix_MSTB:PhoenixContact_MSTBA_2,5_4-G-5,08_1x04_P5.08mm_Horizontal -> powerstep:PhoenixContact_MSTBA_2,5_4-G-5,08_1x04_P5.08mm_Horizontal
Connections:
- wire segments 54 -> 52
- no-connect marks 1 -> 0
Other:
- note added: "en dos conectores para facilitar el \nruteo y que no se pueda conectar la \nalimentacion por error"
- note added: "estoy evaluando no usar agujeros por \nusar montaje sostenido por los \nconectores"
- note added: "segun las pruebas con 200uF \nsera suficiente para un ripple aceptable. \nUso 2 de 100 para que no quede tan alto"
- note removed: "segun las pruebas con 200uF \nsera suficiente para un ripple aceptable\n"

Commit message: achico placa, agrego rj12, defino pistas, ruteo potencia
ahi le voy dando forma. ya rute la potencia y esta mas o menios bien,
ahora estoy viendo el tema de los leds para ponmerlos encima de los
conectores con patas porque es la mejor opcion que se me ocurrio y ya la
tengo probada.. con leds SMD despues tengo que hacer un chino para
sacarlo para afuera y de costado necesito acrilico puro para conducir..
es mas laburo.. con patas hago 2x1.. veremos como queda
Parts:
- removed J2: Conn_01x04, powerstep:PhoenixContact_MSTBA_2,5_4-G-5,08_1x04_P5.08mm_Horizontal, symbol Connector_Generic:Conn_01x04
- added rJ303: RJ12, pap:rj12, symbol pap:RJ12
- C7, C8: footprint powerstep:CP_Radial_D13.0mm_P5.00mm -> pap:CP_Radial_D13.0mm_P5.00mm
- J1, J6: footprint powerstep:PhoenixContact_MSTBA_2,5_2-G-5,08_1x02_P5.08mm_Horizontal -> pap:PhoenixContact_MSTBA_2,5_2-G-5,08_1x02_P5.08mm_Horizontal
- J3: footprint powerstep:PhoenixContact_MSTBA_2,5_4-G-5,08_1x04_P5.08mm_Horizontal -> pap:PhoenixContact_MSTBA_2,5_4-G-5,08_1x04_P5.08mm_Horizontal
- rJ301: footprint pap:rj45_dci -> pap:rj45
- rJ302: footprint powerstep:rj45_dci -> pap:rj45
Connections:
- net labels added: 3V3
- wire segments 52 -> 55
Changed lines of the file:
@@
 EESchema Schematic File Version 4
+LIBS:pap-cache
 EELAYER 26 0
 EELAYER END
@@
 F 0 "J1" H 2030 6500 50  0000 L CNN
 F 1 "Conn_01x02" H 2030 6591 50  0000 L CNN
-F 2 "powerstep:PhoenixContact_MSTBA_2,5_2-G-5,08_1x02_P5.08mm_Horizontal" H 1950 6600 50  0001 C CNN
+F 2 "pap:PhoenixContact_MSTBA_2,5_2-G-5,08_1x02_P5.08mm_Horizontal" H 1950 6600 50  0001 C CNN
 F 3 "~" H 1950 6600 50  0001 C CNN
 	1    1950 6600
@@
 Text HLabel 2350 2850 3    50   Input ~ 0
 SDI
-Text HLabel 7400 1550 2    50   Input ~ 0
+Text HLabel 6650 1800 3    50   Input ~ 0
 Pulse
-Text HLabel 7400 1650 2    50   Input ~ 0
+Text HLabel 6750 1800 3    50   Input ~ 0
 Switch
 Wire Wire Line
@@
 F 0 "J3" H 6120 4267 50  0000 C CNN
 F 1 "Conn_01x04" H 6120 4176 50  0000 C CNN
-F 2 "powerstep:PhoenixContact_MSTBA_2,5_4-G-5,08_1x04_P5.08mm_Horizontal" H 6200 3950 50  0001 C CNN
+F 2 "pap:PhoenixContact_MSTBA_2,5_4-G-5,08_1x04_P5.08mm_Horizontal" H 6200 3950 50  0001 C CNN
 F 3 "~" H 6200 3950 50  0001 C CNN
 	1    6200 3950
@@
 Wire Wire Line
 	2300 6800 2150 6800
-$Comp
-L Connector_Generic:Conn_01x04 J2
-U 1 1 5BC9A7B0
-P 7000 1750
-F 0 "J2" H 6920 1325 50  0000 C CNN
-F 1 "Conn_01x04" H 6920 1416 50  0000 C CNN
-F 2 "powerstep:PhoenixContact_MSTBA_2,5_4-G-5,08_1x04_P5.08mm_Horizontal" H 7000 1750 50  0001 C CNN
-F 3 "~" H 7000 1750 50  0001 C CNN
-	1    7000 1750
-	-1   0    0    1
-$EndComp
-Wire Wire Line
-	7200 1650 7400 1650
-Wire Wire Line
-	7200 1550 7400 1550
 Text HLabel 3600 2850 3    50   Input ~ 0
 SDO
@@
 Text Notes 2000 1050 0    197  ~ 39
 Spi Daisy Chain
-Text Notes 6500 1100 0    197  ~ 39
+Text Notes 7450 1050 0    197  ~ 39
 Paralel Conn\n
 Text Notes 1850 6200 0    197  ~ 39
@@
 F 0 "C7" H 8218 4096 50  0000 L CNN
 F 1 "100uFx100v" V 8200 3850 50  0000 L CNN
-F 2 "powerstep:CP_Radial_D13.0mm_P5.00mm" H 8138 3900 50  0001 C CNN
+F 2 "pap:CP_Radial_D13.0mm_P5.00mm" H 8138 3900 50  0001 C CNN
 F 3 "~" H 8100 4050 50  0001 C CNN
 	1    8100 4050
@@
 Text Notes 7600 4800 0    50   ~ 0
 segun las pruebas con 200uF \nsera suficiente para un ripple aceptable. \nUso 2 de 100 para que no quede tan alto
-Text HLabel 7400 1750 2    50   Input ~ 0
+Text HLabel 6850 1800 3    50   Input ~ 0
 Busy
-Wire Wire Line
-	7400 1750 7200 1750
 Text Notes 7800 1850 0    50   ~ 0
 El busy si se usa como salida para \nmanejar pulso a otro driver es individual
@@
 F 0 "C8" H 8568 4096 50  0000 L CNN
 F 1 "100uFx100v" V 8600 3900 50  0000 L CNN
-F 2 "powerstep:CP_Radial_D13.0mm_P5.00mm" H 8488 3900 50  0001 C CNN
+F 2 "pap:CP_Radial_D13.0mm_P5.00mm" H 8488 3900 50  0001 C CNN
 F 3 "~" H 8450 4050 50  0001 C CNN
 	1    8450 4050
@@
 F 0 "J6" H 2030 6800 50  0000 L CNN
 F 1 "Conn_01x02" H 2030 6891 50  0000 L CNN
-F 2 "powerstep:PhoenixContact_MSTBA_2,5_2-G-5,08_1x02_P5.08mm_Horizontal" H 1950 6900 50  0001 C CNN
+F 2 "pap:PhoenixContact_MSTBA_2,5_2-G-5,08_1x02_P5.08mm_Horizontal" H 1950 6900 50  0001 C CNN
 F 3 "~" H 1950 6900 50  0001 C CNN
 	1    1950 6900
@@
 L pap:G3V3 #PWR0301
 U 1 1 5BB6F1FE
-P 7450 1850
-F 0 "#PWR0301" H 7450 1600 50  0001 C CNN
-F 1 "G3V3" H 7455 1677 50  0000 C CNN
-F 2 "" H 7450 1850 50  0001 C CNN
-F 3 "" H 7450 1850 50  0001 C CNN
-	1    7450 1850
-	1    0    0    -1
-$EndComp
-Wire Wire Line
-	7200 1850 7450 1850
+P 6950 1800
+F 0 "#PWR0301" H 6950 1550 50  0001 C CNN
+F 1 "G3V3" H 6955 1627 50  0000 C CNN
+F 2 "" H 6950 1800 50  0001 C CNN
+F 3 "" H 6950 1800 50  0001 C CNN
+	1    6950 1800
+	1    0    0    -1
+$EndComp
 $Comp
 L pap:RJ45 rJ301
@@
 F 0 "rJ301" V 2541 1220 50  0000 R CNN
 F 1 "RJ45" V 2450 1220 50  0000 R CNN
-F 2 "pap:rj45_dci" V 2550 1675 50  0001 C CNN
+F 2 "pap:rj45" V 2550 1675 50  0001 C CNN
 F 3 "~" V 2550 1675 50  0001 C CNN
 	1    2550 1650
@@
 F 0 "rJ302" V 3791 1220 50  0000 R CNN
 F 1 "RJ45" V 3700 1220 50  0000 R CNN
-F 2 "powerstep:rj45_dci" V 3800 1675 50  0001 C CNN
+F 2 "pap:rj45" V 3800 1675 50  0001 C CNN
 F 3 "~" V 3800 1675 50  0001 C CNN
 	1    3800 1650
@@
 Wire Wire Line
 	6400 4050 6550 4050
+$Comp
+L pap:RJ12 rJ303
+U 1 1 5BB824FD
+P 6750 1200
+F 0 "rJ303" V 6741 870 50  0000 R CNN
+F 1 "RJ12" V 6650 870 50  0000 R CNN
+F 2 "pap:rj12" V 6750 1225 50  0001 C CNN
+F 3 "~" V 6750 1225 50  0001 C CNN
+	1    6750 1200
+	0    -1   -1   0
+$EndComp
+Wire Wire Line
+	6950 1800 6950 1600
+Wire Wire Line
+	6850 1800 6850 1600
+Wire Wire Line
+	6750 1600 6750 1800
+Wire Wire Line
+	6650 1800 6650 1600
+$Comp
+L pap:3V3 #PWR?
+U 1 1 5BB850CF
+P 6250 1800
+AR Path="/5BB850CF" Ref="#PWR?"  Part="1"
+AR Path="/5BA6E8FB/5BB850CF" Ref="#PWR?"  Part="1"
+AR Path="/5BA6E5CE/5BB850CF" Ref="#PWR0110"  Part="1"
+F 0 "#PWR0110" H 6250 1700 50  0001 C CNN
+F 1 "3V3" H 6250 2075 50  0000 C CNN
+F 2 "" H 6250 1800 50  0001 C CNN
+F 3 "" H 6250 1800 50  0001 C CNN
+	1    6250 1800
+	1    0    0    -1
+$EndComp
+Wire Wire Line
+	6450 1600 6450 1850
+Wire Wire Line
+	6450 1850 6250 1850
+Wire Wire Line
+	6250 1800 6250 1850
 $EndSCHEMATC

Commit message: sigo ruteando y acomodando ocsas, agrego algunos leds
Changed lines of the file:
@@
 L pap:G3V3 #PWR0301
 U 1 1 5BB6F1FE
-P 6950 1800
-F 0 "#PWR0301" H 6950 1550 50  0001 C CNN
-F 1 "G3V3" H 6955 1627 50  0000 C CNN
-F 2 "" H 6950 1800 50  0001 C CNN
-F 3 "" H 6950 1800 50  0001 C CNN
-	1    6950 1800
+P 6450 1850
+F 0 "#PWR0301" H 6450 1600 50  0001 C CNN
+F 1 "G3V3" H 6455 1677 50  0000 C CNN
+F 2 "" H 6450 1850 50  0001 C CNN
+F 3 "" H 6450 1850 50  0001 C CNN
+	1    6450 1850
 	1    0    0    -1
 $EndComp
@@
 $EndComp
 Wire Wire Line
-	6950 1800 6950 1600
-Wire Wire Line
 	6850 1800 6850 1600
 Wire Wire Line
@@
 L pap:3V3 #PWR?
 U 1 1 5BB850CF
-P 6250 1800
+P 7150 1800
 AR Path="/5BB850CF" Ref="#PWR?"  Part="1"
 AR Path="/5BA6E8FB/5BB850CF" Ref="#PWR?"  Part="1"
 AR Path="/5BA6E5CE/5BB850CF" Ref="#PWR0110"  Part="1"
-F 0 "#PWR0110" H 6250 1700 50  0001 C CNN
-F 1 "3V3" H 6250 2075 50  0000 C CNN
-F 2 "" H 6250 1800 50  0001 C CNN
-F 3 "" H 6250 1800 50  0001 C CNN
-	1    6250 1800
+F 0 "#PWR0110" H 7150 1700 50  0001 C CNN
+F 1 "3V3" H 7150 2075 50  0000 C CNN
+F 2 "" H 7150 1800 50  0001 C CNN
+F 3 "" H 7150 1800 50  0001 C CNN
+	1    7150 1800
 	1    0    0    -1
 $EndComp
@@
 	6450 1600 6450 1850
 Wire Wire Line
-	6450 1850 6250 1850
+	6950 1850 7150 1850
 Wire Wire Line
-	6250 1800 6250 1850
+	7150 1850 7150 1800
+Wire Wire Line
+	6950 1600 6950 1850
 $EndSCHEMATC

Commit message: ruteo!! no se como pero esta todo conectado!, horrible claro
conecto todo.. bastamte ofiero pero conecto.. y quedan huevos para ir
mejorando.. tampoco esta taaaan mal... y las cosas ya estan en su
lugar.. me quedan varias horas para pulir todo y respetar las reglas de
cada net y demas.. queda un pedazo todavia pero no esta nada mal..
lo que si me di cuenta que estaba pensando mal lo de la cadena de spi y
la de osci, ahora es simple, ficha de in y ficha de out, por la de in
entra sdi y por la de out sale sdo. el ultimo cierra la puerta puentendo
su sdo con un pin suelto de sdo_back que lleva hacia atras el sdo final
y lo termina mandando al uC. o sea es un pin dedicado todo puenteado que
termina en el pin del uC. y para el osci es mas facil porque no necesita
retorno, es una cadena solo de ida, con la salvedad de que por sof,
configuro el primero de la cadena para que genere el osc por sdo y el
segundo mete sdo por el pin de sdi y lo configuro como inversor y asi
siguiendo. no necesita selector de nada, es todo por sof. y despues fui
acomodando un poco el pinout y no mucho mas.. el camino del osci es
larguirucho y lleno de vias pero ese si que quedo atascado y no supe
como sacarlo sin dar una supervuelta.. esperemos que resista..
Parts:
- removed JP301: Clk_Select, Jumper:SolderJumper-3_P2.0mm_Open_TrianglePad1.0x1.5mm, symbol Jumper:Jumper_3_Open
Connections:
- net labels added: Sdo_Back
- net labels removed: Osc, Sdo_Chain
- wire segments 55 -> 50
Changed lines of the file:
@@
 	1    0    0    -1
 $EndComp
+Text HLabel 2750 2850 3    50   Input ~ 0
+CS
 Text HLabel 2150 2850 3    50   Input ~ 0
-CS
+CLK
 Text HLabel 2250 2850 3    50   Input ~ 0
-CLK
-Text HLabel 2350 2850 3    50   Input ~ 0
 SDI
 Text HLabel 6650 1800 3    50   Input ~ 0
 Pulse
-Text HLabel 6750 1800 3    50   Input ~ 0
+Text HLabel 6550 1800 3    50   Input ~ 0
 Switch
 Wire Wire Line
 	2850 2050 2850 2300
 Wire Wire Line
-	2350 2050 2350 2850
+	2350 2050 2350 2550
 $Comp
 L Connector_Generic:Conn_01x04 J3
@@
 Wire Wire Line
 	2300 6800 2150 6800
-Text HLabel 3600 2850 3    50   Input ~ 0
+Text HLabel 3500 2850 3    50   Input ~ 0
 SDO
 Wire Wire Line
-	3600 2050 3600 2850
+	3600 2050 3600 2550
 $Comp
 L pap:G3V3 #PWR0118
@@
 Wire Wire Line
 	4000 2350 4000 2050
-Text HLabel 4350 4750 0    50   Input ~ 0
+Text HLabel 3250 4700 0    50   Input ~ 0
 Busy
 $Comp
 L Jumper:SolderJumper_2_Open JP1
 U 1 1 5BE0DECD
-P 4500 4750
-F 0 "JP1" H 4500 4525 50  0000 C CNN
-F 1 "jumper" H 4500 4616 50  0000 C CNN
-F 2 "Jumper:SolderJumper-2_P1.3mm_Open_RoundedPad1.0x1.5mm" H 4500 4750 50  0001 C CNN
-F 3 "~" H 4500 4750 50  0001 C CNN
-	1    4500 4750
+P 3400 4700
+F 0 "JP1" H 3400 4475 50  0000 C CNN
+F 1 "jumper" H 3400 4566 50  0000 C CNN
+F 2 "Jumper:SolderJumper-2_P1.3mm_Open_RoundedPad1.0x1.5mm" H 3400 4700 50  0001 C CNN
+F 3 "~" H 3400 4700 50  0001 C CNN
+	1    3400 4700
 	-1   0    0    1
 $EndComp
-Text Notes 4200 5200 0    50   ~ 0
+Text Notes 3100 5150 0    50   ~ 0
 si busy va de step, \nno va en cadena SPI, \nsino en conector \nindividual\n
 Wire Wire Line
@@
 	2750 2850 2750 2350
 Connection ~ 2750 2350
-Wire Wire Line
-	2250 2850 2250 2550
 $Comp
 L Device:CP C?
@@
 Text Notes 5900 5000 0    50   ~ 0
 Contemplo doble pin del conector para\npositivo y doble para negativo para \npermitir encadenar alimentacion y/o suplir\nmas corriente\n
-Wire Wire Line
-	2550 2850 2550 2450
 $Comp
 L power:PWR_FLAG #FLG?
@@
 Wire Notes Line
 	5750 2700 5750 5200
-$Comp
-L Jumper:Jumper_3_Open JP?
-U 1 1 5BC3E80A
-P 2500 4850
-AR Path="/5BA6E8FB/5BC3E80A" Ref="JP?"  Part="1"
-AR Path="/5BA6E5CE/5BC3E80A" Ref="JP301"  Part="1"
-F 0 "JP301" V 2546 4937 50  0000 L CNN
-F 1 "Clk_Select" V 2455 4937 50  0000 L CNN
-F 2 "Jumper:SolderJumper-3_P2.0mm_Open_TrianglePad1.0x1.5mm" H 2500 4850 50  0001 C CNN
-F 3 "~" H 2500 4850 50  0001 C CNN
-	1    2500 4850
-	0    -1   -1   0
-$EndComp
-Wire Wire Line
-	2650 4850 2900 4850
-Wire Wire Line
-	2500 4600 2100 4600
-Wire Wire Line
-	2100 5100 2500 5100
-Text HLabel 2100 5100 0    50   Input ~ 0
-Osc_In
-Text HLabel 2100 4600 0    50   Input ~ 0
-Osc_Out
-Text Label 2900 4850 0    50   ~ 0
-Osc
-Text Label 2550 2850 3    50   ~ 0
-Osc
 Text HLabel 2650 2850 3    50   Input ~ 0
 Reset
@@
 Wire Notes Line
 	1200 3900 1200 5300
-Text Notes 2700 5200 0    50   ~ 0
+Text Notes 3900 3200 0    50   ~ 0
 un IC genera y el resto \nconsume CLK y regenera \ninvertido para el siguiente\nCon esto selecciono
 Text Label 2450 2850 3    50   ~ 0
-Sdo_Chain
+Sdo_Back
 Wire Wire Line
 	2850 2300 4100 2300
@@
 	3900 2400 3900 2050
 Wire Wire Line
-	2550 2450 3800 2450
-Connection ~ 2550 2450
-Wire Wire Line
-	2550 2450 2550 2050
-Wire Wire Line
-	3800 2450 3800 2050
-Wire Wire Line
-	2250 2550 3500 2550
-Connection ~ 2250 2550
-Wire Wire Line
-	2250 2550 2250 2050
-Wire Wire Line
-	3500 2550 3500 2050
-Wire Wire Line
-	2150 2600 3400 2600
-Wire Wire Line
-	3400 2600 3400 2050
-Text Label 4650 4750 0    50   ~ 0
+	3500 2850 3500 2050
+Text Label 3550 4700 0    50   ~ 0
 Busy_Out
-Text Label 2750 2850 3    50   ~ 0
+Text Label 2350 2850 3    50   ~ 0
 Busy_Out
 Wire Notes Line
@@
 	2450 2500 2450 2850
 Connection ~ 2450 2500
-Connection ~ 2150 2600
-Wire Wire Line
-	2150 2600 2150 2050
-Wire Wire Line
-	2150 2850 2150 2600
 $Comp
 L Mechanical:MountingHole MH?
@@
 P 6450 1850
 F 0 "#PWR0301" H 6450 1600 50  0001 C CNN
-F 1 "G3V3" H 6455 1677 50  0000 C CNN
+F 1 "G3V3" H 6372 1813 50  0000 R CNN
 F 2 "" H 6450 1850 50  0001 C CNN
 F 3 "" H 6450 1850 50  0001 C CNN
@@
 	6850 1800 6850 1600
 Wire Wire Line
-	6750 1600 6750 1800
+	6550 1600 6550 1800
 Wire Wire Line
 	6650 1800 6650 1600
@@
 Wire Wire Line
 	6950 1600 6950 1850
+Wire Wire Line
+	2150 2050 2150 2600
+Wire Wire Line
+	2350 2550 3600 2550
+Connection ~ 2350 2550
+Wire Wire Line
+	2350 2550 2350 2850
+Wire Wire Line
+	2250 2050 2250 2850
+Wire Wire Line
+	2150 2600 3400 2600
+Connection ~ 2150 2600
+Wire Wire Line
+	2150 2600 2150 2850
+Wire Wire Line
+	3400 2600 3400 2050
+Text HLabel 3800 2850 3    50   Input ~ 0
+Osc_Out
+Wire Wire Line
+	2550 2050 2550 2850
+Wire Wire Line
+	3800 2050 3800 2850
+Text HLabel 2550 2850 3    50   Input ~ 0
+Osc_In
 $EndSCHEMATC
