File: connector.sch (KiCad schematic (older format))
At the start: 12 parts, among them J1 Conn_01x02, J3 Conn_01x04, J6 Conn_01x02

Commit message: sigo ruteando, serigrafia mas gruesa, alineacino etc
Parts:
- D1: footprint Diode_SMD:D_MELF -> pap:D_SMA
- JP1: footprint Jumper:SolderJumper-2_P1.3mm_Open_RoundedPad1.0x1.5mm -> pap:SolderJumper-2_P1.3mm_Open_RoundedPad1.0x1.5mm
- MH301, MH302: footprint MountingHole:MountingHole_3.2mm_M3 -> pap:MountingHole_3.2mm_M3
Changed lines of the file:
@@
 F 0 "D1" V 7604 4129 50  0000 L CNN
 F 1 "SM4007" V 7695 4129 50  0000 L CNN
-F 2 "Diode_SMD:D_MELF" H 7650 3875 50  0001 C CNN
+F 2 "pap:D_SMA" H 7650 3875 50  0001 C CNN
 F 3 "http://cdn-reichelt.de/documents/datenblatt/A400/SMD1N400%23DIO.pdf" H 7650 4050 50  0001 C CNN
 	1    7650 4050
@@
 F 0 "JP1" H 3400 4475 50  0000 C CNN
 F 1 "jumper" H 3400 4566 50  0000 C CNN
-F 2 "Jumper:SolderJumper-2_P1.3mm_Open_RoundedPad1.0x1.5mm" H 3400 4700 50  0001 C CNN
+F 2 "pap:SolderJumper-2_P1.3mm_Open_RoundedPad1.0x1.5mm" H 3400 4700 50  0001 C CNN
 F 3 "~" H 3400 4700 50  0001 C CNN
 	1    3400 4700
@@
 F 0 "MH302" H 4250 6696 50  0000 L CNN
 F 1 "MountingHole" H 4250 6605 50  0000 L CNN
-F 2 "MountingHole:MountingHole_3.2mm_M3" H 4150 6650 50  0001 C CNN
+F 2 "pap:MountingHole_3.2mm_M3" H 4150 6650 50  0001 C CNN
 F 3 "~" H 4150 6650 50  0001 C CNN
 	1    4150 6650
@@
 F 0 "MH301" H 4250 6446 50  0000 L CNN
 F 1 "MountingHole" H 4250 6355 50  0000 L CNN
-F 2 "MountingHole:MountingHole_3.2mm_M3" H 4150 6400 50  0001 C CNN
+F 2 "pap:MountingHole_3.2mm_M3" H 4150 6400 50  0001 C CNN
 F 3 "~" H 4150 6400 50  0001 C CNN
 	1    4150 6400

Commit message: agregando mascaras para alambrado de pistas tie-net,
agregando mascaras para soldar alambres en pistas de potencia, uno con
tie net gnd de 3 con el gnd de 85, tambien agrego planos de tierra para
ambos, y asuntos relacionados con eso. mejor el 3d de las rj;s, agrego
gerbers del fabricante, recien lo veo!! pero se parece bastante a lo que
hice..
Parts:
- added JP301: jumper, pap:SolderJumper-2_P1.3mm_Open_RoundedPad1.0x1.5mm, symbol Jumper:SolderJumper_2_Open
- added NT301, NT?: Net-Tie_2, NetTie:NetTie-2_SMD_Pad0.5mm, symbol Device:Net-Tie_2
Connections:
- wire segments 50 -> 58
Other:
- note added: "Contemplo doble pin del conector \npara positivo y doble para \nnegativo para permitir \nencadenar alimentacion y/o \nsuplir mas corriente\n"
- note added: "Se conectan desde 2 \npines de g3v3 a \n1 de g85v\n"
- note added: "con este puente se evita \nel uso de un stub externo"
- note added: "proteccion inversion \nde polaridad\n"
- note added: "segun pruebas 200uF es \nsuficiente Uso 2 de 100 \npara que no quede tan alto"
- note removed: "Contemplo doble pin del conector para\npositivo y doble para negativo para \npermitir encadenar alimentacion y/o suplir\nmas corriente\n"
- note removed: "segun las pruebas con 200uF \nsera suficiente para un ripple aceptable. \nUso 2 de 100 para que no quede tan alto"
Changed lines of the file:
@@
 L Device:CP C?
 U 1 1 5BDFE583
-P 8100 4050
+P 9550 4050
 AR Path="/5BA6E8FB/5BDFE583" Ref="C?"  Part="1"
 AR Path="/5BA6E5CE/5BDFE583" Ref="C7"  Part="1"
-F 0 "C7" H 8218 4096 50  0000 L CNN
-F 1 "100uFx100v" V 8200 3850 50  0000 L CNN
-F 2 "pap:CP_Radial_D13.0mm_P5.00mm" H 8138 3900 50  0001 C CNN
-F 3 "~" H 8100 4050 50  0001 C CNN
-	1    8100 4050
+F 0 "C7" H 9668 4096 50  0000 L CNN
+F 1 "100uFx100v" V 9650 3850 50  0000 L CNN
+F 2 "pap:CP_Radial_D13.0mm_P5.00mm" H 9588 3900 50  0001 C CNN
+F 3 "~" H 9550 4050 50  0001 C CNN
+	1    9550 4050
 	1    0    0    -1
 $EndComp
@@
 L pap:85V #PWR?
 U 1 1 5BDFE58A
-P 8100 3900
+P 9550 3900
 AR Path="/5BDFE58A" Ref="#PWR?"  Part="1"
 AR Path="/5BA6E8FB/5BDFE58A" Ref="#PWR?"  Part="1"
 AR Path="/5BA6E5CE/5BDFE58A" Ref="#PWR0101"  Part="1"
-F 0 "#PWR0101" H 8100 3800 50  0001 C CNN
-F 1 "85V" H 8100 4175 50  0000 C CNN
-F 2 "" H 8100 3900 50  0001 C CNN
-F 3 "" H 8100 3900 50  0001 C CNN
-	1    8100 3900
+F 0 "#PWR0101" H 9550 3800 50  0001 C CNN
+F 1 "85V" H 9550 4175 50  0000 C CNN
+F 2 "" H 9550 3900 50  0001 C CNN
+F 3 "" H 9550 3900 50  0001 C CNN
+	1    9550 3900
 	1    0    0    -1
 $EndComp
@@
 L pap:G85V #PWR?
 U 1 1 5BDFE590
-P 8100 4200
+P 9550 4200
 AR Path="/5BDFE590" Ref="#PWR?"  Part="1"
 AR Path="/5BA6E8FB/5BDFE590" Ref="#PWR?"  Part="1"
 AR Path="/5BA6E5CE/5BDFE590" Ref="#PWR0102"  Part="1"
-F 0 "#PWR0102" H 8100 3950 50  0001 C CNN
-F 1 "G85V" H 8105 4027 50  0000 C CNN
-F 2 "" H 8100 4200 50  0001 C CNN
-F 3 "" H 8100 4200 50  0001 C CNN
-	1    8100 4200
+F 0 "#PWR0102" H 9550 3950 50  0001 C CNN
+F 1 "G85V" H 9555 4027 50  0000 C CNN
+F 2 "" H 9550 4200 50  0001 C CNN
+F 3 "" H 9550 4200 50  0001 C CNN
+	1    9550 4200
 	1    0    0    -1
 $EndComp
@@
 Text Notes 7800 1650 0    50   ~ 0
 El fin de carrera y el step es individual \npor modulo asi que va por fuera \nde la cadena SPI\n
-Text Notes 7600 4800 0    50   ~ 0
-segun las pruebas con 200uF \nsera suficiente para un ripple aceptable. \nUso 2 de 100 para que no quede tan alto
+Text Notes 9300 4750 0    50   ~ 0
+segun pruebas 200uF es \nsuficiente Uso 2 de 100 \npara que no quede tan alto
 Text HLabel 6850 1800 3    50   Input ~ 0
 Busy
@@
 Wire Wire Line
 	4000 2350 4000 2050
-Text HLabel 3250 4700 0    50   Input ~ 0
+Text HLabel 1750 4650 0    50   Input ~ 0
 Busy
 $Comp
 L Jumper:SolderJumper_2_Open JP1
 U 1 1 5BE0DECD
-P 3400 4700
-F 0 "JP1" H 3400 4475 50  0000 C CNN
-F 1 "jumper" H 3400 4566 50  0000 C CNN
-F 2 "pap:SolderJumper-2_P1.3mm_Open_RoundedPad1.0x1.5mm" H 3400 4700 50  0001 C CNN
-F 3 "~" H 3400 4700 50  0001 C CNN
-	1    3400 4700
+P 1900 4650
+F 0 "JP1" H 1900 4425 50  0000 C CNN
+F 1 "jumper" H 1900 4516 50  0000 C CNN
+F 2 "pap:SolderJumper-2_P1.3mm_Open_RoundedPad1.0x1.5mm" H 1900 4650 50  0001 C CNN
+F 3 "~" H 1900 4650 50  0001 C CNN
+	1    1900 4650
 	-1   0    0    1
 $EndComp
-Text Notes 3100 5150 0    50   ~ 0
+Text Notes 1600 5100 0    50   ~ 0
 si busy va de step, \nno va en cadena SPI, \nsino en conector \nindividual\n
 Wire Wire Line
@@
 L Device:CP C?
 U 1 1 5BE152B2
-P 8450 4050
+P 9900 4050
 AR Path="/5BA6E8FB/5BE152B2" Ref="C?"  Part="1"
 AR Path="/5BA6E5CE/5BE152B2" Ref="C8"  Part="1"
-F 0 "C8" H 8568 4096 50  0000 L CNN
-F 1 "100uFx100v" V 8600 3900 50  0000 L CNN
-F 2 "pap:CP_Radial_D13.0mm_P5.00mm" H 8488 3900 50  0001 C CNN
-F 3 "~" H 8450 4050 50  0001 C CNN
-	1    8450 4050
+F 0 "C8" H 10018 4096 50  0000 L CNN
+F 1 "100uFx100v" V 10050 3900 50  0000 L CNN
+F 2 "pap:CP_Radial_D13.0mm_P5.00mm" H 9938 3900 50  0001 C CNN
+F 3 "~" H 9900 4050 50  0001 C CNN
+	1    9900 4050
 	1    0    0    -1
 $EndComp
@@
 L pap:85V #PWR?
 U 1 1 5BE152B8
-P 8450 3900
+P 9900 3900
 AR Path="/5BE152B8" Ref="#PWR?"  Part="1"
 AR Path="/5BA6E8FB/5BE152B8" Ref="#PWR?"  Part="1"
 AR Path="/5BA6E5CE/5BE152B8" Ref="#PWR0103"  Part="1"
-F 0 "#PWR0103" H 8450 3800 50  0001 C CNN
-F 1 "85V" H 8450 4175 50  0000 C CNN
-F 2 "" H 8450 3900 50  0001 C CNN
-F 3 "" H 8450 3900 50  0001 C CNN
-	1    8450 3900
+F 0 "#PWR0103" H 9900 3800 50  0001 C CNN
+F 1 "85V" H 9900 4175 50  0000 C CNN
+F 2 "" H 9900 3900 50  0001 C CNN
+F 3 "" H 9900 3900 50  0001 C CNN
+	1    9900 3900
 	1    0    0    -1
 $EndComp
@@
 L pap:G85V #PWR?
 U 1 1 5BE152BE
-P 8450 4200
+P 9900 4200
 AR Path="/5BE152BE" Ref="#PWR?"  Part="1"
 AR Path="/5BA6E8FB/5BE152BE" Ref="#PWR?"  Part="1"
 AR Path="/5BA6E5CE/5BE152BE" Ref="#PWR0104"  Part="1"
-F 0 "#PWR0104" H 8450 3950 50  0001 C CNN
-F 1 "G85V" H 8455 4027 50  0000 C CNN
-F 2 "" H 8450 4200 50  0001 C CNN
-F 3 "" H 8450 4200 50  0001 C CNN
-	1    8450 4200
+F 0 "#PWR0104" H 9900 3950 50  0001 C CNN
+F 1 "G85V" H 9905 4027 50  0000 C CNN
+F 2 "" H 9900 4200 50  0001 C CNN
+F 3 "" H 9900 4200 50  0001 C CNN
+	1    9900 4200
 	1    0    0    -1
 $EndComp
@@
 Connection ~ 6550 4150
 Text Notes 5900 5000 0    50   ~ 0
-Contemplo doble pin del conector para\npositivo y doble para negativo para \npermitir encadenar alimentacion y/o suplir\nmas corriente\n
+Contemplo doble pin del conector \npara positivo y doble para \nnegativo para permitir \nencadenar alimentacion y/o \nsuplir mas corriente\n
 $Comp
 L power:PWR_FLAG #FLG?
@@
 $EndComp
 Wire Notes Line
-	5750 5200 9350 5200
-Wire Notes Line
-	9350 5200 9350 2700
-Wire Notes Line
-	9350 2700 5750 2700
+	5750 5200 10500 5200
+Wire Notes Line
+	10500 5200 10500 2700
+Wire Notes Line
+	10500 2700 5750 2700
 Wire Notes Line
 	5750 2700 5750 5200
@@
 Wire Wire Line
 	2650 2850 2650 2400
-Text Notes 2450 4250 0    197  ~ 39
+Text Notes 1950 4200 0    197  ~ 39
 Pins Selector
 Wire Notes Line
@@
 Wire Wire Line
 	3500 2850 3500 2050
-Text Label 3550 4700 0    50   ~ 0
+Text Label 2050 4650 0    50   ~ 0
 Busy_Out
 Text Label 2350 2850 3    50   ~ 0
@@
 Text HLabel 2550 2850 3    50   Input ~ 0
 Osc_In
+$Comp
+L Jumper:SolderJumper_2_Open JP301
+U 1 1 5BC269EF
+P 3800 4700
+F 0 "JP301" H 3800 4475 50  0000 C CNN
+F 1 "jumper" H 3800 4566 50  0000 C CNN
+F 2 "pap:SolderJumper-2_P1.3mm_Open_RoundedPad1.0x1.5mm" H 3800 4700 50  0001 C CNN
+F 3 "~" H 3800 4700 50  0001 C CNN
+	1    3800 4700
+	-1   0    0    1
+$EndComp
+Text Notes 3350 4950 0    50   ~ 0
+con este puente se evita \nel uso de un stub externo
+Text HLabel 3950 4700 2    50   Input ~ 0
+SDO
+Text Label 3650 4700 2    50   ~ 0
+Sdo_Back
+Text Notes 7400 4700 0    50   ~ 0
+proteccion inversion \nde polaridad\n
+$Comp
+L pap:G85V #PWR?
+U 1 1 5BCA053C
+P 8400 4200
+AR Path="/5BCA053C" Ref="#PWR?"  Part="1"
+AR Path="/5BA6E8FB/5BCA053C" Ref="#PWR?"  Part="1"
+AR Path="/5BA6E5CE/5BCA053C" Ref="#PWR0114"  Part="1"
+F 0 "#PWR0114" H 8400 3950 50  0001 C CNN
+F 1 "G85V" H 8405 4027 50  0000 C CNN
+F 2 "" H 8400 4200 50  0001 C CNN
+F 3 "" H 8400 4200 50  0001 C CNN
+	1    8400 4200
+	1    0    0    -1
+$EndComp
+$Comp
+L pap:G3V3 #PWR0117
+U 1 1 5BCA06DC
+P 8700 4200
+F 0 "#PWR0117" H 8700 3950 50  0001 C CNN
+F 1 "G3V3" H 8705 4027 50  0000 C CNN
+F 2 "" H 8700 4200 50  0001 C CNN
+F 3 "" H 8700 4200 50  0001 C CNN
+	1    8700 4200
+	-1   0    0    -1
+$EndComp
+$Comp
+L Device:Net-Tie_2 NT301
+U 1 1 5BCA0988
+P 8550 3900
+F 0 "NT301" H 8550 4078 50  0000 C CNN
+F 1 "Net-Tie_2" H 8550 3987 50  0000 C CNN
+F 2 "NetTie:NetTie-2_SMD_Pad0.5mm" H 8550 3900 50  0001 C CNN
+F 3 "~" H 8550 3900 50  0001 C CNN
+	1    8550 3900
+	1    0    0    -1
+$EndComp
+Wire Wire Line
+	8400 4200 8400 3900
+Wire Wire Line
+	8400 3900 8450 3900
+Wire Wire Line
+	8700 3900 8700 4200
+Wire Wire Line
+	8700 3900 8650 3900
+$Comp
+L Device:Net-Tie_2 NT?
+U 1 1 5BCA6648
+P 8550 3550
+F 0 "NT?" H 8550 3728 50  0000 C CNN
+F 1 "Net-Tie_2" H 8550 3637 50  0000 C CNN
+F 2 "NetTie:NetTie-2_SMD_Pad0.5mm" H 8550 3550 50  0001 C CNN
+F 3 "~" H 8550 3550 50  0001 C CNN
+	1    8550 3550
+	1    0    0    -1
+$EndComp
+Wire Wire Line
+	8450 3550 8400 3550
+Wire Wire Line
+	8400 3550 8400 3900
+Connection ~ 8400 3900
+Wire Wire Line
+	8650 3550 8700 3550
+Wire Wire Line
+	8700 3550 8700 3900
+Connection ~ 8700 3900
+Text Notes 8300 4800 0    50   ~ 0
+Se conectan desde 2 \npines de g3v3 a \n1 de g85v\n
 $EndSCHEMATC

Commit message: cambio de nombres, mejorop serigrafia, agrego pin
agrego el pin de flag ya que me sobraba un pin en el RJ12, cambio los
nombres de 0-50 para motor y 51 a 100 para conector, ajusto el espesor
de la seri, y algunas cosas mas..
Parts:
- NT51: renamed from NT?; footprint NetTie:NetTie-2_SMD_Pad0.5mm -> pap:NetTie-2_SMD_Pad0.2mm_sin_seri
- NT52: renamed from NT301; footprint NetTie:NetTie-2_SMD_Pad0.5mm -> pap:NetTie-2_SMD_Pad0.2mm_sin_seri
- renumbered C7 to C51, C8 to C52, D1 to D51, J3 to J51, J1 to J52, J6 to J53, rJ301 to J54, rJ302 to J55, rJ303 to J56, JP1 to JP51, JP301 to JP52, MH301 to MH51, MH302 to MH52
Connections:
- net labels added: Flag
- wire segments 58 -> 59
Other:
- note added: "Pins Select"
- note removed: "Pins Selector"
Changed lines of the file:
@@
 $EndDescr
 $Comp
-L Connector_Generic:Conn_01x02 J1
+L Connector_Generic:Conn_01x02 J52
 U 1 1 5BA7B68B
 P 1950 6600
-F 0 "J1" H 2030 6500 50  0000 L CNN
+F 0 "J52" H 2030 6500 50  0000 L CNN
 F 1 "Conn_01x02" H 2030 6591 50  0000 L CNN
 F 2 "pap:PhoenixContact_MSTBA_2,5_2-G-5,08_1x02_P5.08mm_Horizontal" H 1950 6600 50  0001 C CNN
@@
 	6550 3850 6550 3700
 $Comp
-L Diode:SM4007 D1
+L Diode:SM4007 D51
 U 1 1 5BA7B8EB
 P 7650 4050
-F 0 "D1" V 7604 4129 50  0000 L CNN
+F 0 "D51" V 7604 4129 50  0000 L CNN
 F 1 "SM4007" V 7695 4129 50  0000 L CNN
 F 2 "pap:D_SMA" H 7650 3875 50  0001 C CNN
@@
 	2350 2050 2350 2550
 $Comp
-L Connector_Generic:Conn_01x04 J3
+L Connector_Generic:Conn_01x04 J51
 U 1 1 5BC94397
 P 6200 3950
-F 0 "J3" H 6120 4267 50  0000 C CNN
+F 0 "J51" H 6120 4267 50  0000 C CNN
 F 1 "Conn_01x04" H 6120 4176 50  0000 C CNN
 F 2 "pap:PhoenixContact_MSTBA_2,5_4-G-5,08_1x04_P5.08mm_Horizontal" H 6200 3950 50  0001 C CNN
@@
 P 9550 4050
 AR Path="/5BA6E8FB/5BDFE583" Ref="C?"  Part="1"
-AR Path="/5BA6E5CE/5BDFE583" Ref="C7"  Part="1"
-F 0 "C7" H 9668 4096 50  0000 L CNN
-F 1 "100uFx100v" V 9650 3850 50  0000 L CNN
+AR Path="/5BA6E5CE/5BDFE583" Ref="C51"  Part="1"
+F 0 "C51" H 9432 4096 50  0000 R CNN
+F 1 "100uFx100v" H 9432 4005 50  0000 R CNN
 F 2 "pap:CP_Radial_D13.0mm_P5.00mm" H 9588 3900 50  0001 C CNN
 F 3 "~" H 9550 4050 50  0001 C CNN
@@
 Busy
 $Comp
-L Jumper:SolderJumper_2_Open JP1
+L Jumper:SolderJumper_2_Open JP51
 U 1 1 5BE0DECD
 P 1900 4650
-F 0 "JP1" H 1900 4425 50  0000 C CNN
+F 0 "JP51" H 1900 4425 50  0000 C CNN
 F 1 "jumper" H 1900 4516 50  0000 C CNN
 F 2 "pap:SolderJumper-2_P1.3mm_Open_RoundedPad1.0x1.5mm" H 1900 4650 50  0001 C CNN
@@
 P 9900 4050
 AR Path="/5BA6E8FB/5BE152B2" Ref="C?"  Part="1"
-AR Path="/5BA6E5CE/5BE152B2" Ref="C8"  Part="1"
-F 0 "C8" H 10018 4096 50  0000 L CNN
-F 1 "100uFx100v" V 10050 3900 50  0000 L CNN
+AR Path="/5BA6E5CE/5BE152B2" Ref="C52"  Part="1"
+F 0 "C52" H 10018 4096 50  0000 L CNN
+F 1 "100uFx100v" H 10018 4005 50  0000 L CNN
 F 2 "pap:CP_Radial_D13.0mm_P5.00mm" H 9938 3900 50  0001 C CNN
 F 3 "~" H 9900 4050 50  0001 C CNN
@@
 $EndComp
 $Comp
-L Connector_Generic:Conn_01x02 J6
+L Connector_Generic:Conn_01x02 J53
 U 1 1 5BE15A46
 P 1950 6900
-F 0 "J6" H 2030 6800 50  0000 L CNN
+F 0 "J53" H 2030 6800 50  0000 L CNN
 F 1 "Conn_01x02" H 2030 6891 50  0000 L CNN
 F 2 "pap:PhoenixContact_MSTBA_2,5_2-G-5,08_1x02_P5.08mm_Horizontal" H 1950 6900 50  0001 C CNN
@@
 Wire Wire Line
 	2650 2850 2650 2400
-Text Notes 1950 4200 0    197  ~ 39
-Pins Selector
+Text Notes 2150 4250 0    197  ~ 39
+Pins Select
 Wire Notes Line
 	1100 3650 5250 3650
@@
 P 4150 6650
 AR Path="/5BB850B6" Ref="MH?"  Part="1"
-AR Path="/5BA6E5CE/5BB850B6" Ref="MH302"  Part="1"
-F 0 "MH302" H 4250 6696 50  0000 L CNN
+AR Path="/5BA6E5CE/5BB850B6" Ref="MH52"  Part="1"
+F 0 "MH52" H 4250 6696 50  0000 L CNN
 F 1 "MountingHole" H 4250 6605 50  0000 L CNN
 F 2 "pap:MountingHole_3.2mm_M3" H 4150 6650 50  0001 C CNN
@@
 P 4150 6400
 AR Path="/5BB850BD" Ref="MH?"  Part="1"
-AR Path="/5BA6E5CE/5BB850BD" Ref="MH301"  Part="1"
-F 0 "MH301" H 4250 6446 50  0000 L CNN
+AR Path="/5BA6E5CE/5BB850BD" Ref="MH51"  Part="1"
+F 0 "MH51" H 4250 6446 50  0000 L CNN
 F 1 "MountingHole" H 4250 6355 50  0000 L CNN
 F 2 "pap:MountingHole_3.2mm_M3" H 4150 6400 50  0001 C CNN
@@
 $EndComp
 $Comp
-L pap:RJ45 rJ301
+L pap:RJ45 J54
 U 1 1 5BB97209
 P 2550 1650
-F 0 "rJ301" V 2541 1220 50  0000 R CNN
+F 0 "J54" V 2541 1220 50  0000 R CNN
 F 1 "RJ45" V 2450 1220 50  0000 R CNN
 F 2 "pap:rj45" V 2550 1675 50  0001 C CNN
@@
 $EndComp
 $Comp
-L pap:RJ45 rJ302
+L pap:RJ45 J55
 U 1 1 5BB97330
 P 3800 1650
-F 0 "rJ302" V 3791 1220 50  0000 R CNN
+F 0 "J55" V 3791 1220 50  0000 R CNN
 F 1 "RJ45" V 3700 1220 50  0000 R CNN
 F 2 "pap:rj45" V 3800 1675 50  0001 C CNN
@@
 Wire Wire Line
 	6400 4050 6550 4050
-$Comp
-L pap:RJ12 rJ303
-U 1 1 5BB824FD
-P 6750 1200
-F 0 "rJ303" V 6741 870 50  0000 R CNN
-F 1 "RJ12" V 6650 870 50  0000 R CNN
-F 2 "pap:rj12" V 6750 1225 50  0001 C CNN
-F 3 "~" V 6750 1225 50  0001 C CNN
-	1    6750 1200
-	0    -1   -1   0
-$EndComp
 Wire Wire Line
 	6850 1800 6850 1600
@@
 Osc_In
 $Comp
-L Jumper:SolderJumper_2_Open JP301
+L Jumper:SolderJumper_2_Open JP52
 U 1 1 5BC269EF
 P 3800 4700
-F 0 "JP301" H 3800 4475 50  0000 C CNN
+F 0 "JP52" H 3800 4475 50  0000 C CNN
 F 1 "jumper" H 3800 4566 50  0000 C CNN
 F 2 "pap:SolderJumper-2_P1.3mm_Open_RoundedPad1.0x1.5mm" H 3800 4700 50  0001 C CNN
@@
 $EndComp
 $Comp
-L Device:Net-Tie_2 NT301
+L Device:Net-Tie_2 NT52
 U 1 1 5BCA0988
 P 8550 3900
-F 0 "NT301" H 8550 4078 50  0000 C CNN
+F 0 "NT52" H 8550 4078 50  0000 C CNN
 F 1 "Net-Tie_2" H 8550 3987 50  0000 C CNN
-F 2 "NetTie:NetTie-2_SMD_Pad0.5mm" H 8550 3900 50  0001 C CNN
+F 2 "pap:NetTie-2_SMD_Pad0.2mm_sin_seri" H 8550 3900 50  0001 C CNN
 F 3 "~" H 8550 3900 50  0001 C CNN
 	1    8550 3900
@@
 	8700 3900 8650 3900
 $Comp
-L Device:Net-Tie_2 NT?
+L Device:Net-Tie_2 NT51
 U 1 1 5BCA6648
 P 8550 3550
-F 0 "NT?" H 8550 3728 50  0000 C CNN
+F 0 "NT51" H 8550 3728 50  0000 C CNN
 F 1 "Net-Tie_2" H 8550 3637 50  0000 C CNN
-F 2 "NetTie:NetTie-2_SMD_Pad0.5mm" H 8550 3550 50  0001 C CNN
+F 2 "pap:NetTie-2_SMD_Pad0.2mm_sin_seri" H 8550 3550 50  0001 C CNN
 F 3 "~" H 8550 3550 50  0001 C CNN
 	1    8550 3550
@@
 Text Notes 8300 4800 0    50   ~ 0
 Se conectan desde 2 \npines de g3v3 a \n1 de g85v\n
+Text HLabel 6750 1800 3    50   Input ~ 0
+Flag
+$Comp
+L pap:RJ12 J56
+U 1 1 5BB824FD
+P 6750 1200
+F 0 "J56" V 6741 870 50  0000 R CNN
+F 1 "RJ12" V 6650 870 50  0000 R CNN
+F 2 "pap:rj12" V 6750 1225 50  0001 C CNN
+F 3 "~" V 6750 1225 50  0001 C CNN
+	1    6750 1200
+	0    -1   -1   0
+$EndComp
+Wire Wire Line
+	6750 1800 6750 1600
 $EndSCHEMATC

Commit message: aghrego serigrafia, logos, faltan fiduciales aun
Parts:
- removed MH51, MH52: MountingHole, pap:MountingHole_3.2mm_M3, symbol Mechanical:MountingHole
Other:
- note removed: "Holes"
- note removed: "estoy evaluando no usar agujeros por \nusar montaje sostenido por los \nconectores"
Changed lines of the file:
@@
 $Descr A4 11693 8268
 encoding utf-8
-Sheet 3 3
+Sheet 3 4
 Title "PaP"
 Date "2018-09-21"
@@
 Connection ~ 2450 2500
 $Comp
-L Mechanical:MountingHole MH?
-U 1 1 5BB850B6
-P 4150 6650
-AR Path="/5BB850B6" Ref="MH?"  Part="1"
-AR Path="/5BA6E5CE/5BB850B6" Ref="MH52"  Part="1"
-F 0 "MH52" H 4250 6696 50  0000 L CNN
-F 1 "MountingHole" H 4250 6605 50  0000 L CNN
-F 2 "pap:MountingHole_3.2mm_M3" H 4150 6650 50  0001 C CNN
-F 3 "~" H 4150 6650 50  0001 C CNN
-	1    4150 6650
-	1    0    0    -1
-$EndComp
-$Comp
-L Mechanical:MountingHole MH?
-U 1 1 5BB850BD
-P 4150 6400
-AR Path="/5BB850BD" Ref="MH?"  Part="1"
-AR Path="/5BA6E5CE/5BB850BD" Ref="MH51"  Part="1"
-F 0 "MH51" H 4250 6446 50  0000 L CNN
-F 1 "MountingHole" H 4250 6355 50  0000 L CNN
-F 2 "pap:MountingHole_3.2mm_M3" H 4150 6400 50  0001 C CNN
-F 3 "~" H 4150 6400 50  0001 C CNN
-	1    4150 6400
-	1    0    0    -1
-$EndComp
-Text Notes 4000 6100 0    197  ~ 39
-Holes
-Wire Notes Line
-	3700 7350 5200 7350
-Wire Notes Line
-	5200 7350 5200 5650
-Wire Notes Line
-	5200 5650 3700 5650
-Wire Notes Line
-	3700 5650 3700 7350
-$Comp
 L pap:G3V3 #PWR0301
 U 1 1 5BB6F1FE
@@
 Text Notes 1600 7250 0    50   ~ 0
 en dos conectores para facilitar el \nruteo y que no se pueda conectar la \nalimentacion por error
-Text Notes 3750 7150 0    50   ~ 0
-estoy evaluando no usar agujeros por \nusar montaje sostenido por los \nconectores
 Wire Wire Line
 	6550 4150 6750 4150
