File: motor.sch (KiCad schematic (older format))
At the start: 33 parts

Commit message: agrego mas conectores y paso a pcb (todo mal!)
agregue conectores RJ45 para el encadenamiento spi y busyflag, pero no
para pulse.. es lo voy a mandar aparte porque es individual por cada
driver.. al igual que switch, y vere si alguna cosa mas.. en el rj me
sobran aun 2 pines.. ya vere que mando..lastima que no puedo mandar
pulse por ahi.. porque al ser 1 por driver necesito ir directo desde el
controlador.. sino como?... pase a pcb para ver que onda nada mas y
obvio me faltan definir los footprints de casi todo.. pero al menos
paso...orcad ya estaria llorando y no podria hacer nada...como sea, esta
bueno...sigo
Parts:
- removed R? (x3): R, symbol Device:R
- added D4: LED, LED_SMD:LED_0805_2012Metric, symbol Device:LED
- added R1, R8: R, symbol Device:R
- gave numbers to parts that had none: 30
Connections:
- net labels removed: clk_in, clk_out
- wire segments 221 -> 226

Commit message: armo huella step01 y asigno casi todas las huellas
ahi hice el landpattern del steo01, que es un parto, pero quedo bueno..
al tiempo que aprendi a editar y la verdad es que es comodo.. me animo a
decir que supera a allegro, y de hecho se parece demasiado en muchas
cosas.. huele a copia de algun lado.. incluiso los nombres en los menus
son iguales... como sea, ya quedo eso, lo que si tuve que volar algunos
pines repetidos en el simbolo porque sino era un chino tener muchos
pines repetidos, o sea en la huella tengo un pin que va a parar a
multiples pines en el esquemativo. si bien lo logre hacer superponiendo
encimados los pines en el esquemativo y dejandolos invisibles excepto
uno, eso funca, pero es un azco... preferi volar todos y dejar la union
univoca y listo.. al simbolo le faltan pines, pero el landpattern no los
necesita porque se unen todos en una misma masa de pad. despues pase
todas las huellas del resto del chiquitaje y ademas acomodo los power
netlist que estaban mal y de paso voy puliendo el disenio en general..
va quedando.. un poco mas y paso a tirar pista
Parts:
- removed C7: 220uFx100v, symbol Device:CP
- removed R5: R, symbol Device:R
- added D12: D_Zener, Diode_SMD:D_MiniMELF, symbol Device:D_Zener
- C1, C2, C3, C4, C5, C6: footprint (none) -> Capacitor_SMD:C_0805_2012Metric
- R1, R10, R11, R12, R13, R14, R2, R6, R7, R8, R9: footprint (none) -> Resistor_SMD:R_0805_2012Metric
- R3, R4: footprint (none) -> Resistor_SMD:R_1812_4532Metric_Pad1.30x3.40mm_HandSolder
- U1: footprint (none) -> powerstep:powerstep
- Y1: footprint (none) -> Crystal:Crystal_HC49-U_Vertical
Connections:
- net labels removed: 100V
- wire segments 226 -> 137
Other:
- note added: "Contemplo leds para ver movimiento en \nsincro con el motor mas algunos de debug \ncomo flag\n"
- note added: "Controlador PaP"
- note added: "Leds debug\n"
- note added: "Protecciones\n"
- note added: "Recomiendan un diodo \ndesde 3 a 15 en inversa.\n"
- note added: "idealmente 32Mhz, pero \npodria ir tambien 16\n \n"
- moved on the sheet: D9

Commit message: arranco a rutear, cambio xtal por SMD y opcion CLKIN
arranque a tirar pist porque me estaba aburriendo ya, de paso voy
practivcando los shortcuts y demas.. esta muy copado y te aviso.. es
plagio a allegro.. no cabe dudas.. como sea, cambie el Xtal por uno SMD
de 4 pines que se consigue y minimiza el espacio, agegue tambien clkin
para mandar clk a todos por igual con el PWM del uC para sincronizar con
un selector para poder usar el xtal si es que el PWM se pierde por
fanout o ruido.. y no mucho mas
Parts:
- removed Y1: 32Mhz, Crystal:Crystal_HC49-U_Vertical, symbol Device:Crystal
- added JP2: Clk_Select, Jumper:SolderJumper-3_P2.0mm_Open_TrianglePad1.0x1.5mm, symbol Jumper:Jumper_3_Open
- added Y1: 32Mhz, Crystal:Crystal_SMD_2016-4Pin_2.0x1.6mm, symbol Device:Crystal_GND23
Connections:
- net labels added: CLKIN
- net labels removed: G15V
- wire segments 137 -> 148
Other:
- note removed: "idealmente 32Mhz, pero \npodria ir tambien 16\n \n"

Commit message: Cambio Rj's vuela xtal, entra Reset, agrego tornillos
Hago de todo un poco entre lo que saco el xtal porque ya probe que no se
necesita, elijo un IC que gnere 16Mhz y lo encadeno al resto, el RJ lo
cambie por otra que se parece mas a la que voy a usar, pero hay que
verificar, agregue un selector de osc, y agregue unos agujeros de
tornillos que no se si los quiero. va bien.. tengo que meterle mas al
ruteo
Parts:
- removed C2, C3: 10pF, Capacitor_SMD:C_0805_2012Metric, symbol Device:C
- removed JP2: Clk_Select, Jumper:SolderJumper-3_P2.0mm_Open_TrianglePad1.0x1.5mm, symbol Jumper:Jumper_3_Open
- removed R1, R2: R, Resistor_SMD:R_0805_2012Metric, symbol Device:R
- removed Y1: 32Mhz, Crystal:Crystal_SMD_2016-4Pin_2.0x1.6mm, symbol Device:Crystal_GND23
- added D201: LL4148, Diode_SMD:D_MiniMELF, symbol Diode:LL4148
- added D202: LED, LED_SMD:LED_0805_2012Metric, symbol Device:LED
- added R201, R202: R, Resistor_SMD:R_0805_2012Metric, symbol Device:R
Connections:
- net labels added: Adc, Osc_In, Osc_Out, Switch_Local, flag
- net labels removed: CLKIN
- wire segments 148 -> 134
Other:
- note added: "Dejo un diodo para evitar \naccidentes al conectar. \nsi mandan 85v no pasa nada. \nEl pin ya tienen pullup"
- note added: "El IC tiene Pull down, con esto \narrancaria encendido o lo controlo\ncon el pin externo"
- note added: "Filter and Protections"
- note added: "Motor Driver IC"
- note added: "Se usa para compensar \npotencia"
- note removed: "Controlador PaP"
- note removed: "Protecciones\n"
- moved on the sheet: D9

Commit message: cambio nombres, hago board edge, defino capas, posicion y demas
hice de todo un poco, principalmente le di forma a la placa con una
dimensino pasable, ajuste los conectores que aun no me convencen, pero
cambie la entrada para el conector de 4 y los motores en 2 de 2, cosa
que la alimentacion este toda en un solo conector y me queda piola para
que los motores salgan del IC para los costados. en cuanto a la logica
aun no me decido si voy a poner otra RJ para la salida d busy y demas o
meto bornera.. estouy mas del lado de la RJ y me quedaria genial para
poner los leds arriba de la RJ o a un costado.. puedo elegir eso.. mepa
que vamos con eso y asi no hay manera de mezclar fichas tampoco, porque
pongo un 6P6C RJ12 y ya.. hasta me sobran 2 pines.. bueno despues lo
sigo.
Parts:
- R3, R4: footprint Resistor_SMD:R_1812_4532Metric_Pad1.30x3.40mm_HandSolder -> Resistor_SMD:R_2816_7142Metric_Pad3.20x4.45mm_HandSolder
- U1: footprint powerstep:powerstep -> pap:powerstep; symbol schematic.lib:powerstep01 -> pap:powerstep01
Changed lines of the file:
@@
 EESchema Schematic File Version 4
-LIBS:pap-cache
 EELAYER 26 0
 EELAYER END
@@
 	8950 3600 8800 3600
 $Comp
-L schematic.lib:85V #PWR?
+L pap:85V #PWR?
 U 1 1 5BA6F2D7
 P 9400 3600
@@
 	8800 4400 8800 3950
 $Comp
-L schematic.lib:85V #PWR?
+L pap:85V #PWR?
 U 1 1 5BA70B2F
 P 8400 3600
@@
 	7000 4000 7150 4000
 $Comp
-L schematic.lib:3V3 #PWR?
+L pap:3V3 #PWR?
 U 1 1 5BA71FD4
 P 8200 3600
@@
 Connection ~ 10350 8800
 $Comp
-L schematic.lib:85V #PWR?
+L pap:85V #PWR?
 U 1 1 5BA7823D
 P 10350 8400
@@
 $EndComp
 $Comp
-L schematic.lib:G85V #PWR?
+L pap:G85V #PWR?
 U 1 1 5BA78330
 P 10350 9250
@@
 $EndComp
 $Comp
-L schematic.lib:G85V #PWR?
+L pap:G85V #PWR?
 U 1 1 5BA7866F
 P 10700 9250
@@
 Connection ~ 5750 6250
 $Comp
-L schematic.lib:G85V #PWR?
+L pap:G85V #PWR?
 U 1 1 5BAB2AA9
 P 7350 3400
@@
 F 0 "R4" H 5120 6696 50  0000 L CNN
 F 1 "R" H 5120 6605 50  0000 L CNN
-F 2 "Resistor_SMD:R_1812_4532Metric_Pad1.30x3.40mm_HandSolder" V 4980 6650 50  0001 C CNN
+F 2 "Resistor_SMD:R_2816_7142Metric_Pad3.20x4.45mm_HandSolder" V 4980 6650 50  0001 C CNN
 F 3 "~" H 5050 6650 50  0001 C CNN
 	1    5050 6650
@@
 Connection ~ 5050 6050
 $Comp
-L schematic.lib:G85V #PWR?
+L pap:G85V #PWR?
 U 1 1 5BB52220
 P 5050 6850
@@
 F 0 "R3" H 4870 1396 50  0000 L CNN
 F 1 "R" H 4870 1305 50  0000 L CNN
-F 2 "Resistor_SMD:R_1812_4532Metric_Pad1.30x3.40mm_HandSolder" V 4730 1350 50  0001 C CNN
+F 2 "Resistor_SMD:R_2816_7142Metric_Pad3.20x4.45mm_HandSolder" V 4730 1350 50  0001 C CNN
 F 3 "~" H 4800 1350 50  0001 C CNN
 	1    4800 1350
@@
 $EndComp
 $Comp
-L schematic.lib:G85V #PWR?
+L pap:G85V #PWR?
 U 1 1 5BC3AA66
 P 4800 1550
@@
 	3150 3600 2650 3600
 $Comp
-L schematic.lib:3V3 #PWR?
+L pap:3V3 #PWR?
 U 1 1 5BDAFBFA
 P 2100 3900
@@
 	3150 3900 2100 3900
 $Comp
-L schematic.lib:G3V3 #PWR?
+L pap:G3V3 #PWR?
 U 1 1 5BDFC6AD
 P 1850 3400
@@
 	3150 3400 1850 3400
 $Comp
-L schematic.lib:G3V3 #PWR?
+L pap:G3V3 #PWR?
 U 1 1 5BE572B5
 P 2500 4700
@@
 	7000 3600 7600 3600
 $Comp
-L schematic.lib:15V #PWR?
+L pap:15V #PWR?
 U 1 1 5BEEBABF
 P 8600 3600
@@
 $EndComp
 $Comp
-L schematic.lib:3V3 #PWR?
+L pap:3V3 #PWR?
 U 1 1 5C13AF57
 P 2250 8650
@@
 $EndComp
 $Comp
-L schematic.lib:3V3 #PWR?
+L pap:3V3 #PWR?
 U 1 1 5C1814CA
 P 2650 8650
@@
 MotorA2
 $Comp
-L schematic.lib:G85V #PWR?
+L pap:G85V #PWR?
 U 1 1 5C1E693B
 P 3050 9300
@@
 $EndComp
 $Comp
-L schematic.lib:G85V #PWR?
+L pap:G85V #PWR?
 U 1 1 5C1E6A5E
 P 3450 9300
@@
 MotorB2
 $Comp
-L schematic.lib:G85V #PWR?
+L pap:G85V #PWR?
 U 1 1 5C1E6CFF
 P 3850 9300
@@
 $EndComp
 $Comp
-L schematic.lib:G85V #PWR?
+L pap:G85V #PWR?
 U 1 1 5C1E6D05
 P 4250 9300
@@
 	6800 9150 6800 8800
 $Comp
-L schematic.lib:3V3 #PWR?
+L pap:3V3 #PWR?
 U 1 1 5C2DB7F9
 P 6500 8800
@@
 $EndComp
 $Comp
-L schematic.lib:15V #PWR?
+L pap:15V #PWR?
 U 1 1 5C2F89A6
 P 6800 8800
@@
 $EndComp
 $Comp
-L schematic.lib:3V3 #PWR?
+L pap:3V3 #PWR?
 U 1 1 5BA82210
 P 1850 8650
@@
 	4250 9250 4250 9300
 $Comp
-L schematic.lib:85V #PWR?
+L pap:85V #PWR?
 U 1 1 5BCCC35B
 P 6050 1750
@@
 $EndComp
 $Comp
-L schematic.lib:85V #PWR?
+L pap:85V #PWR?
 U 1 1 5BCDA53A
 P 4100 1750
@@
 $EndComp
 $Comp
-L schematic.lib:85V #PWR?
+L pap:85V #PWR?
 U 1 1 5BCE8ABD
 P 3850 6800
@@
 $EndComp
 $Comp
-L schematic.lib:85V #PWR?
+L pap:85V #PWR?
 U 1 1 5BCF752D
 P 6350 6750
@@
 	8600 3600 8600 4000
 $Comp
-L schematic.lib:powerstep01 U1
+L pap:powerstep01 U1
 U 1 1 5BA75207
 P 5050 4100
 F 0 "U1" H 3650 6000 50  0000 C CNN
 F 1 "powerstep01" H 3550 6100 50  0000 C CNN
-F 2 "powerstep:powerstep" H 4150 3600 50  0001 C CNN
+F 2 "pap:powerstep" H 4150 3600 50  0001 C CNN
 F 3 "" H 3250 6150 50  0001 C CNN
 	1    5050 4100
@@
 $EndComp
 $Comp
-L schematic.lib:G85V #PWR?
+L pap:G85V #PWR?
 U 1 1 5BDAC7A4
 P 11000 9250
@@
 	7150 4000 8600 4000
 $Comp
-L schematic.lib:G85V #PWR?
+L pap:G85V #PWR?
 U 1 1 5BB5D627
 P 7300 4100
@@
 Switch
 $Comp
-L schematic.lib:G3V3 #PWR?
+L pap:G3V3 #PWR?
 U 1 1 5BBB31C8
 P 7950 9100
@@
 $EndComp
 $Comp
-L schematic.lib:3V3 #PWR?
+L pap:3V3 #PWR?
 U 1 1 5BBC458D
 P 9350 8800
@@
 	1400 9250 1400 9350
 $Comp
-L schematic.lib:85V #PWR?
+L pap:85V #PWR?
 U 1 1 5BB57E18
 P 1400 8650
@@
 $EndComp
 $Comp
-L schematic.lib:G85V #PWR?
+L pap:G85V #PWR?
 U 1 1 5BB583DF
 P 1400 9350
@@
 Wire Notes Line
 	1150 850  1150 7200
-Connection ~ 8800 3750
 Wire Wire Line
 	8800 3750 8800 3950

Commit message: achico placa, agrego rj12, defino pistas, ruteo potencia
ahi le voy dando forma. ya rute la potencia y esta mas o menios bien,
ahora estoy viendo el tema de los leds para ponmerlos encima de los
conectores con patas porque es la mejor opcion que se me ocurrio y ya la
tengo probada.. con leds SMD despues tengo que hacer un chino para
sacarlo para afuera y de costado necesito acrilico puro para conducir..
es mas laburo.. con patas hago 2x1.. veremos como queda
Connections:
- net labels added: Cpump, SenseA, SenseB, Vboot, Vs
Changed lines of the file:
@@
 EESchema Schematic File Version 4
+LIBS:pap-cache
 EELAYER 26 0
 EELAYER END
@@
 AR Path="/5BA6E8FB/5BB5D627" Ref="#PWR0107"  Part="1"
 F 0 "#PWR0107" H 7300 3850 50  0001 C CNN
-F 1 "G85V" H 7305 3927 50  0000 C CNN
+F 1 "G85V" H 7388 4063 50  0000 L CNN
 F 2 "" H 7300 4100 50  0001 C CNN
 F 3 "" H 7300 4100 50  0001 C CNN
@@
 Wire Wire Line
 	8800 3600 8800 3950
+Text Label 4650 6400 0    50   ~ 0
+SenseA
+Text Label 4450 1150 0    50   ~ 0
+SenseB
+Text Label 8000 4400 0    50   ~ 0
+Vboot
+Text Label 8000 4500 0    50   ~ 0
+Vs
+Text Label 8000 4300 0    50   ~ 0
+Cpump
 $EndSCHEMATC

Commit message: sigo ruteando y acomodando ocsas, agrego algunos leds
Parts:
- D10, D11, D202, D7, D8: footprint LED_SMD:LED_0805_2012Metric -> pap:led5p_enchufable
- D4, D5, D6: footprint LED_SMD:LED_0805_2012Metric -> pap:led5p_rj
Changed lines of the file:
@@
 F 0 "D5" V 2288 8683 50  0000 R CNN
 F 1 "LED" V 2197 8683 50  0000 R CNN
-F 2 "LED_SMD:LED_0805_2012Metric" H 2250 8800 50  0001 C CNN
+F 2 "pap:led5p_rj" H 2250 8800 50  0001 C CNN
 F 3 "~" H 2250 8800 50  0001 C CNN
 	1    2250 8800
@@
 F 0 "D6" V 2688 8683 50  0000 R CNN
 F 1 "LED" V 2597 8683 50  0000 R CNN
-F 2 "LED_SMD:LED_0805_2012Metric" H 2650 8800 50  0001 C CNN
+F 2 "pap:led5p_rj" H 2650 8800 50  0001 C CNN
 F 3 "~" H 2650 8800 50  0001 C CNN
 	1    2650 8800
@@
 F 0 "D7" V 3088 8683 50  0000 R CNN
 F 1 "LED" V 2997 8683 50  0000 R CNN
-F 2 "LED_SMD:LED_0805_2012Metric" H 3050 8800 50  0001 C CNN
+F 2 "pap:led5p_enchufable" H 3050 8800 50  0001 C CNN
 F 3 "~" H 3050 8800 50  0001 C CNN
 	1    3050 8800
@@
 F 0 "D8" V 3488 8683 50  0000 R CNN
 F 1 "LED" V 3397 8683 50  0000 R CNN
-F 2 "LED_SMD:LED_0805_2012Metric" H 3450 8800 50  0001 C CNN
+F 2 "pap:led5p_enchufable" H 3450 8800 50  0001 C CNN
 F 3 "~" H 3450 8800 50  0001 C CNN
 	1    3450 8800
@@
 F 0 "D10" V 3888 8683 50  0000 R CNN
 F 1 "LED" V 3797 8683 50  0000 R CNN
-F 2 "LED_SMD:LED_0805_2012Metric" H 3850 8800 50  0001 C CNN
+F 2 "pap:led5p_enchufable" H 3850 8800 50  0001 C CNN
 F 3 "~" H 3850 8800 50  0001 C CNN
 	1    3850 8800
@@
 F 0 "D11" V 4288 8683 50  0000 R CNN
 F 1 "LED" V 4197 8683 50  0000 R CNN
-F 2 "LED_SMD:LED_0805_2012Metric" H 4250 8800 50  0001 C CNN
+F 2 "pap:led5p_enchufable" H 4250 8800 50  0001 C CNN
 F 3 "~" H 4250 8800 50  0001 C CNN
 	1    4250 8800
@@
 F 0 "D4" V 1888 8683 50  0000 R CNN
 F 1 "LED" V 1797 8683 50  0000 R CNN
-F 2 "LED_SMD:LED_0805_2012Metric" H 1850 8800 50  0001 C CNN
+F 2 "pap:led5p_rj" H 1850 8800 50  0001 C CNN
 F 3 "~" H 1850 8800 50  0001 C CNN
 	1    1850 8800
@@
 L Device:LED D202
 U 1 1 5BB4DB4E
-P 1400 8800
-F 0 "D202" V 1438 8683 50  0000 R CNN
-F 1 "LED" V 1347 8683 50  0000 R CNN
-F 2 "LED_SMD:LED_0805_2012Metric" H 1400 8800 50  0001 C CNN
-F 3 "~" H 1400 8800 50  0001 C CNN
-	1    1400 8800
+P 4600 8800
+F 0 "D202" V 4638 8683 50  0000 R CNN
+F 1 "LED" V 4547 8683 50  0000 R CNN
+F 2 "pap:led5p_enchufable" H 4600 8800 50  0001 C CNN
+F 3 "~" H 4600 8800 50  0001 C CNN
+	1    4600 8800
 	0    -1   -1   0
 $EndComp
@@
 L Device:R R202
 U 1 1 5BB4DB5B
-P 1400 9100
-F 0 "R202" H 1330 9054 50  0000 R CNN
-F 1 "R" H 1330 9145 50  0000 R CNN
-F 2 "Resistor_SMD:R_0805_2012Metric" V 1330 9100 50  0001 C CNN
-F 3 "~" H 1400 9100 50  0001 C CNN
-	1    1400 9100
-	-1   0    0    1
-$EndComp
-Wire Wire Line
-	1400 9250 1400 9350
+P 4600 9100
+F 0 "R202" H 4530 9054 50  0000 R CNN
+F 1 "R" H 4530 9145 50  0000 R CNN
+F 2 "Resistor_SMD:R_0805_2012Metric" V 4530 9100 50  0001 C CNN
+F 3 "~" H 4600 9100 50  0001 C CNN
+	1    4600 9100
+	-1   0    0    1
+$EndComp
+Wire Wire Line
+	4600 9250 4600 9350
 $Comp
 L pap:85V #PWR?
 U 1 1 5BB57E18
-P 1400 8650
+P 4600 8650
 AR Path="/5BB57E18" Ref="#PWR?"  Part="1"
 AR Path="/5BA6E8FB/5BB57E18" Ref="#PWR0201"  Part="1"
-F 0 "#PWR0201" H 1400 8550 50  0001 C CNN
-F 1 "85V" H 1400 8925 50  0000 C CNN
-F 2 "" H 1400 8650 50  0001 C CNN
-F 3 "" H 1400 8650 50  0001 C CNN
-	1    1400 8650
+F 0 "#PWR0201" H 4600 8550 50  0001 C CNN
+F 1 "85V" H 4600 8925 50  0000 C CNN
+F 2 "" H 4600 8650 50  0001 C CNN
+F 3 "" H 4600 8650 50  0001 C CNN
+	1    4600 8650
 	1    0    0    -1
 $EndComp
@@
 L pap:G85V #PWR?
 U 1 1 5BB583DF
-P 1400 9350
+P 4600 9350
 AR Path="/5BB583DF" Ref="#PWR?"  Part="1"
 AR Path="/5BA6E8FB/5BB583DF" Ref="#PWR0202"  Part="1"
-F 0 "#PWR0202" H 1400 9100 50  0001 C CNN
-F 1 "G85V" H 1405 9177 50  0000 C CNN
-F 2 "" H 1400 9350 50  0001 C CNN
-F 3 "" H 1400 9350 50  0001 C CNN
-	1    1400 9350
-	1    0    0    -1
-$EndComp
+F 0 "#PWR0202" H 4600 9100 50  0001 C CNN
+F 1 "G85V" H 4605 9177 50  0000 C CNN
+F 2 "" H 4600 9350 50  0001 C CNN
+F 3 "" H 4600 9350 50  0001 C CNN
+	1    4600 9350
+	1    0    0    -1
+$EndComp

Commit message: ruteo!! no se como pero esta todo conectado!, horrible claro
conecto todo.. bastamte ofiero pero conecto.. y quedan huevos para ir
mejorando.. tampoco esta taaaan mal... y las cosas ya estan en su
lugar.. me quedan varias horas para pulir todo y respetar las reglas de
cada net y demas.. queda un pedazo todavia pero no esta nada mal..
lo que si me di cuenta que estaba pensando mal lo de la cadena de spi y
la de osci, ahora es simple, ficha de in y ficha de out, por la de in
entra sdi y por la de out sale sdo. el ultimo cierra la puerta puentendo
su sdo con un pin suelto de sdo_back que lleva hacia atras el sdo final
y lo termina mandando al uC. o sea es un pin dedicado todo puenteado que
termina en el pin del uC. y para el osci es mas facil porque no necesita
retorno, es una cadena solo de ida, con la salvedad de que por sof,
configuro el primero de la cadena para que genere el osc por sdo y el
segundo mete sdo por el pin de sdi y lo configuro como inversor y asi
siguiendo. no necesita selector de nada, es todo por sof. y despues fui
acomodando un poco el pinout y no mucho mas.. el camino del osci es
larguirucho y lleno de vias pero ese si que quedo atascado y no supe
como sacarlo sin dar una supervuelta.. esperemos que resista..
Parts:
- removed D10, D202, D8: LED, pap:led5p_enchufable, symbol Device:LED
- added D10, D202, D8: LED_I, pap:led5p_enchufable, symbol pap:LED_I
- added D203, D204: LED, pap:led5p_rj, symbol Device:LED
- added R203, R204: R, Resistor_SMD:R_0805_2012Metric, symbol Device:R
- C4, C5: footprint Capacitor_SMD:C_0805_2012Metric -> Capacitor_SMD:C_1206_3216Metric_Pad1.42x1.75mm_HandSolder
Connections:
- net labels removed: flag
- wire segments 134 -> 136
