File: motor.sch (KiCad schematic (older format))
At the start: 35 parts, among them U1 powerstep01

Commit message: sigo ruteando, serigrafia mas gruesa, alineacino etc
Parts:
- C1, C6: footprint Capacitor_SMD:C_0805_2012Metric -> pap:C_0805_2012Metric
- C4, C5: footprint Capacitor_SMD:C_1206_3216Metric_Pad1.42x1.75mm_HandSolder -> pap:C_1206_3216Metric_Pad1.42x1.75mm_HandSolder
- D12, D2, D201, D3: footprint Diode_SMD:D_MiniMELF -> pap:D_MiniMELF
- D9: footprint Diode_SMD:D_MELF -> pap:D_SMA
- R10, R11, R12, R13, R14, R201, R202, R203, R204, R6, R7, R8, R9: footprint Resistor_SMD:R_0805_2012Metric -> pap:R_0805_2012Metric
- R3, R4: footprint Resistor_SMD:R_2816_7142Metric_Pad3.20x4.45mm_HandSolder -> pap:R_2816_7142Metric_Pad3.20x4.45mm_HandSolder
Changed lines of the file:
@@
 F 0 "D2" H 8950 4166 50  0000 C CNN
 F 1 "LL4148" H 8950 4075 50  0000 C CNN
-F 2 "Diode_SMD:D_MiniMELF" H 8950 3775 50  0001 C CNN
+F 2 "pap:D_MiniMELF" H 8950 3775 50  0001 C CNN
 F 3 "http://www.vishay.com/docs/85557/ll4148.pdf" H 8950 3950 50  0001 C CNN
 	1    8950 3950
@@
 F 0 "D3" H 9250 4166 50  0000 C CNN
 F 1 "LL4148" H 9250 4075 50  0000 C CNN
-F 2 "Diode_SMD:D_MiniMELF" H 9250 3775 50  0001 C CNN
+F 2 "pap:D_MiniMELF" H 9250 3775 50  0001 C CNN
 F 3 "http://www.vishay.com/docs/85557/ll4148.pdf" H 9250 3950 50  0001 C CNN
 	1    9250 3950
@@
 F 0 "C5" H 8985 4054 50  0000 R CNN
 F 1 "C" H 8985 4145 50  0000 R CNN
-F 2 "Capacitor_SMD:C_1206_3216Metric_Pad1.42x1.75mm_HandSolder" H 9138 3950 50  0001 C CNN
+F 2 "pap:C_1206_3216Metric_Pad1.42x1.75mm_HandSolder" H 9138 3950 50  0001 C CNN
 F 3 "~" H 9100 4100 50  0001 C CNN
 	1    9100 4100
@@
 F 0 "C4" V 9352 3600 50  0000 C CNN
 F 1 "C" V 9261 3600 50  0000 C CNN
-F 2 "Capacitor_SMD:C_1206_3216Metric_Pad1.42x1.75mm_HandSolder" H 9138 3450 50  0001 C CNN
+F 2 "pap:C_1206_3216Metric_Pad1.42x1.75mm_HandSolder" H 9138 3450 50  0001 C CNN
 F 3 "~" H 9100 3600 50  0001 C CNN
 	1    9100 3600
@@
 F 0 "R6" H 10420 8646 50  0000 L CNN
 F 1 "R" H 10420 8555 50  0000 L CNN
-F 2 "Resistor_SMD:R_0805_2012Metric" V 10280 8600 50  0001 C CNN
+F 2 "pap:R_0805_2012Metric" V 10280 8600 50  0001 C CNN
 F 3 "~" H 10350 8600 50  0001 C CNN
 	1    10350 8600
@@
 F 0 "R7" H 10420 9096 50  0000 L CNN
 F 1 "R" H 10420 9005 50  0000 L CNN
-F 2 "Resistor_SMD:R_0805_2012Metric" V 10280 9050 50  0001 C CNN
+F 2 "pap:R_0805_2012Metric" V 10280 9050 50  0001 C CNN
 F 3 "~" H 10350 9050 50  0001 C CNN
 	1    10350 9050
@@
 F 0 "C6" H 10585 8954 50  0000 R CNN
 F 1 "C" H 10585 9045 50  0000 R CNN
-F 2 "Capacitor_SMD:C_0805_2012Metric" H 10738 8850 50  0001 C CNN
+F 2 "pap:C_0805_2012Metric" H 10738 8850 50  0001 C CNN
 F 3 "~" H 10700 9000 50  0001 C CNN
 	1    10700 9000
@@
 F 0 "R4" H 5120 6696 50  0000 L CNN
 F 1 "R" H 5120 6605 50  0000 L CNN
-F 2 "Resistor_SMD:R_2816_7142Metric_Pad3.20x4.45mm_HandSolder" V 4980 6650 50  0001 C CNN
+F 2 "pap:R_2816_7142Metric_Pad3.20x4.45mm_HandSolder" V 4980 6650 50  0001 C CNN
 F 3 "~" H 5050 6650 50  0001 C CNN
 	1    5050 6650
@@
 F 0 "R3" H 4870 1396 50  0000 L CNN
 F 1 "R" H 4870 1305 50  0000 L CNN
-F 2 "Resistor_SMD:R_2816_7142Metric_Pad3.20x4.45mm_HandSolder" V 4730 1350 50  0001 C CNN
+F 2 "pap:R_2816_7142Metric_Pad3.20x4.45mm_HandSolder" V 4730 1350 50  0001 C CNN
 F 3 "~" H 4800 1350 50  0001 C CNN
 	1    4800 1350
@@
 F 0 "R9" H 2030 9054 50  0000 R CNN
 F 1 "R" H 2030 9145 50  0000 R CNN
-F 2 "Resistor_SMD:R_0805_2012Metric" V 2030 9100 50  0001 C CNN
+F 2 "pap:R_0805_2012Metric" V 2030 9100 50  0001 C CNN
 F 3 "~" H 2100 9100 50  0001 C CNN
 	1    2100 9100
@@
 F 0 "R10" H 1330 9054 50  0000 R CNN
 F 1 "R" H 1330 9145 50  0000 R CNN
-F 2 "Resistor_SMD:R_0805_2012Metric" V 1330 9100 50  0001 C CNN
+F 2 "pap:R_0805_2012Metric" V 1330 9100 50  0001 C CNN
 F 3 "~" H 1400 9100 50  0001 C CNN
 	1    1400 9100
@@
 F 0 "R11" H 2930 9054 50  0000 R CNN
 F 1 "R" H 2930 9145 50  0000 R CNN
-F 2 "Resistor_SMD:R_0805_2012Metric" V 2930 9100 50  0001 C CNN
+F 2 "pap:R_0805_2012Metric" V 2930 9100 50  0001 C CNN
 F 3 "~" H 3000 9100 50  0001 C CNN
 	1    3000 9100
@@
 F 0 "R12" H 3330 9054 50  0000 R CNN
 F 1 "R" H 3330 9145 50  0000 R CNN
-F 2 "Resistor_SMD:R_0805_2012Metric" V 3330 9100 50  0001 C CNN
+F 2 "pap:R_0805_2012Metric" V 3330 9100 50  0001 C CNN
 F 3 "~" H 3400 9100 50  0001 C CNN
 	1    3400 9100
@@
 F 0 "R13" H 3730 9054 50  0000 R CNN
 F 1 "R" H 3730 9145 50  0000 R CNN
-F 2 "Resistor_SMD:R_0805_2012Metric" V 3730 9100 50  0001 C CNN
+F 2 "pap:R_0805_2012Metric" V 3730 9100 50  0001 C CNN
 F 3 "~" H 3800 9100 50  0001 C CNN
 	1    3800 9100
@@
 F 0 "R14" H 4130 9054 50  0000 R CNN
 F 1 "R" H 4130 9145 50  0000 R CNN
-F 2 "Resistor_SMD:R_0805_2012Metric" V 4130 9100 50  0001 C CNN
+F 2 "pap:R_0805_2012Metric" V 4130 9100 50  0001 C CNN
 F 3 "~" H 4200 9100 50  0001 C CNN
 	1    4200 9100
@@
 F 0 "D9" V 6546 8871 50  0000 R CNN
 F 1 "SM4007" V 6455 8871 50  0000 R CNN
-F 2 "Diode_SMD:D_MELF" H 6500 8775 50  0001 C CNN
+F 2 "pap:D_SMA" H 6500 8775 50  0001 C CNN
 F 3 "http://cdn-reichelt.de/documents/datenblatt/A400/SMD1N400%23DIO.pdf" H 6500 8950 50  0001 C CNN
 	1    6500 8950
@@
 F 0 "R8" H 930 9054 50  0000 R CNN
 F 1 "R" H 930 9145 50  0000 R CNN
-F 2 "Resistor_SMD:R_0805_2012Metric" V 930 9100 50  0001 C CNN
+F 2 "pap:R_0805_2012Metric" V 930 9100 50  0001 C CNN
 F 3 "~" H 1000 9100 50  0001 C CNN
 	1    1000 9100
@@
 F 0 "D12" V 10954 9079 50  0000 L CNN
 F 1 "D_Zener" V 11045 9079 50  0000 L CNN
-F 2 "Diode_SMD:D_MiniMELF" H 11000 9000 50  0001 C CNN
+F 2 "pap:D_MiniMELF" H 11000 9000 50  0001 C CNN
 F 3 "~" H 11000 9000 50  0001 C CNN
 	1    11000 9000
@@
 F 0 "C1" H 7835 8904 50  0000 R CNN
 F 1 "C" H 7835 8995 50  0000 R CNN
-F 2 "Capacitor_SMD:C_0805_2012Metric" H 7988 8800 50  0001 C CNN
+F 2 "pap:C_0805_2012Metric" H 7988 8800 50  0001 C CNN
 F 3 "~" H 7950 8950 50  0001 C CNN
 	1    7950 8950
@@
 F 0 "R201" V 9150 9000 50  0000 C CNN
 F 1 "R" V 9250 9000 50  0000 C CNN
-F 2 "Resistor_SMD:R_0805_2012Metric" V 9280 9000 50  0001 C CNN
+F 2 "pap:R_0805_2012Metric" V 9280 9000 50  0001 C CNN
 F 3 "~" H 9350 9000 50  0001 C CNN
 	1    9350 9000
@@
 F 0 "D201" H 8250 8866 50  0000 C CNN
 F 1 "LL4148" H 8250 8775 50  0000 C CNN
-F 2 "Diode_SMD:D_MiniMELF" H 8250 8475 50  0001 C CNN
+F 2 "pap:D_MiniMELF" H 8250 8475 50  0001 C CNN
 F 3 "http://www.vishay.com/docs/85557/ll4148.pdf" H 8250 8650 50  0001 C CNN
 	1    8250 8650
@@
 F 0 "R202" H 4530 9004 50  0000 R CNN
 F 1 "R" H 4530 9095 50  0000 R CNN
-F 2 "Resistor_SMD:R_0805_2012Metric" V 4530 9050 50  0001 C CNN
+F 2 "pap:R_0805_2012Metric" V 4530 9050 50  0001 C CNN
 F 3 "~" H 4600 9050 50  0001 C CNN
 	1    4600 9050
@@
 F 0 "R203" H 1680 9054 50  0000 R CNN
 F 1 "R" H 1680 9145 50  0000 R CNN
-F 2 "Resistor_SMD:R_0805_2012Metric" V 1680 9100 50  0001 C CNN
+F 2 "pap:R_0805_2012Metric" V 1680 9100 50  0001 C CNN
 F 3 "~" H 1750 9100 50  0001 C CNN
 	1    1750 9100
@@
 F 0 "R204" H 2380 9054 50  0000 R CNN
 F 1 "R" H 2380 9145 50  0000 R CNN
-F 2 "Resistor_SMD:R_0805_2012Metric" V 2380 9100 50  0001 C CNN
+F 2 "pap:R_0805_2012Metric" V 2380 9100 50  0001 C CNN
 F 3 "~" H 2450 9100 50  0001 C CNN
 	1    2450 9100

Commit message: agregando mascaras para alambrado de pistas tie-net,
agregando mascaras para soldar alambres en pistas de potencia, uno con
tie net gnd de 3 con el gnd de 85, tambien agrego planos de tierra para
ambos, y asuntos relacionados con eso. mejor el 3d de las rj;s, agrego
gerbers del fabricante, recien lo veo!! pero se parece bastante a lo que
hice..
Parts:
- removed D9: SM4007, pap:D_SMA, symbol Diode:SM4007
- added D205, D206: LL4148, pap:D_MiniMELF, symbol Diode:LL4148
Connections:
- wire segments 136 -> 143
Other:
- note added: "Recomiendan low drop diodo \ndesde 3 a 15 y 15 a 85 en inversa.\nVer powerstep datasheet Pag. 36 \n"
- note removed: "Recomiendan un diodo \ndesde 3 a 15 en inversa.\n"
Changed lines of the file:
@@
 	1    0    0    -1
 $EndComp
-$Comp
-L Diode:SM4007 D9
-U 1 1 5C1F5B94
-P 6500 8950
-F 0 "D9" V 6546 8871 50  0000 R CNN
-F 1 "SM4007" V 6455 8871 50  0000 R CNN
-F 2 "pap:D_SMA" H 6500 8775 50  0001 C CNN
-F 3 "http://cdn-reichelt.de/documents/datenblatt/A400/SMD1N400%23DIO.pdf" H 6500 8950 50  0001 C CNN
-	1    6500 8950
-	0    -1   -1   0
-$EndComp
-Wire Wire Line
-	6500 9150 6800 9150
-Wire Wire Line
-	6800 9150 6800 8800
+Wire Wire Line
+	5900 9150 6200 9150
+Wire Wire Line
+	6200 9150 6200 8650
 $Comp
 L pap:3V3 #PWR?
 U 1 1 5C2DB7F9
-P 6500 8800
+P 5900 8550
 AR Path="/5C2DB7F9" Ref="#PWR?"  Part="1"
 AR Path="/5BA6E8FB/5C2DB7F9" Ref="#PWR0152"  Part="1"
-F 0 "#PWR0152" H 6500 8700 50  0001 C CNN
-F 1 "3V3" H 6500 9075 50  0000 C CNN
-F 2 "" H 6500 8800 50  0001 C CNN
-F 3 "" H 6500 8800 50  0001 C CNN
-	1    6500 8800
+F 0 "#PWR0152" H 5900 8450 50  0001 C CNN
+F 1 "3V3" H 5900 8825 50  0000 C CNN
+F 2 "" H 5900 8550 50  0001 C CNN
+F 3 "" H 5900 8550 50  0001 C CNN
+	1    5900 8550
 	1    0    0    -1
 $EndComp
@@
 L pap:15V #PWR?
 U 1 1 5C2F89A6
-P 6800 8800
+P 6200 8550
 AR Path="/5C2F89A6" Ref="#PWR?"  Part="1"
 AR Path="/5BA6E8FB/5C2F89A6" Ref="#PWR0153"  Part="1"
-F 0 "#PWR0153" H 6800 8700 50  0001 C CNN
-F 1 "15V" H 6800 9075 50  0000 C CNN
-F 2 "" H 6800 8800 50  0001 C CNN
-F 3 "" H 6800 8800 50  0001 C CNN
-	1    6800 8800
-	1    0    0    -1
-$EndComp
-Wire Wire Line
-	6500 9150 6500 9100
+F 0 "#PWR0153" H 6200 8450 50  0001 C CNN
+F 1 "15V" H 6200 8825 50  0000 C CNN
+F 2 "" H 6200 8550 50  0001 C CNN
+F 3 "" H 6200 8550 50  0001 C CNN
+	1    6200 8550
+	1    0    0    -1
+$EndComp
+Wire Wire Line
+	5900 9150 5900 9050
 Wire Wire Line
 	1400 9250 1400 9350
@@
 Text Notes 2250 9850 0    50   ~ 0
 Contemplo leds para ver movimiento en \nsincro con el motor mas algunos de debug \ncomo flag\n
-Text Notes 6200 9550 0    50   ~ 0
-Recomiendan un diodo \ndesde 3 a 15 en inversa.\n
+Text Notes 5750 9600 0    50   ~ 0
+Recomiendan low drop diodo \ndesde 3 a 15 y 15 a 85 en inversa.\nVer powerstep datasheet Pag. 36 \n
 $Comp
 L Device:D_Zener D12
@@
 	0    -1   -1   0
 $EndComp
+$Comp
+L Diode:LL4148 D?
+U 1 1 5BC459B0
+P 5900 8900
+AR Path="/5BC459B0" Ref="D?"  Part="1"
+AR Path="/5BA6E8FB/5BC459B0" Ref="D205"  Part="1"
+F 0 "D205" V 5946 8821 50  0000 R CNN
+F 1 "LL4148" V 5855 8821 50  0000 R CNN
+F 2 "pap:D_MiniMELF" H 5900 8725 50  0001 C CNN
+F 3 "http://www.vishay.com/docs/85557/ll4148.pdf" H 5900 8900 50  0001 C CNN
+	1    5900 8900
+	0    -1   -1   0
+$EndComp
+$Comp
+L pap:85V #PWR?
+U 1 1 5BC5A76A
+P 6600 8550
+AR Path="/5BC5A76A" Ref="#PWR?"  Part="1"
+AR Path="/5BA6E8FB/5BC5A76A" Ref="#PWR0113"  Part="1"
+F 0 "#PWR0113" H 6600 8450 50  0001 C CNN
+F 1 "85V" H 6600 8825 50  0000 C CNN
+F 2 "" H 6600 8550 50  0001 C CNN
+F 3 "" H 6600 8550 50  0001 C CNN
+	1    6600 8550
+	1    0    0    -1
+$EndComp
+$Comp
+L Diode:LL4148 D?
+U 1 1 5BC5A9C8
+P 6400 8900
+AR Path="/5BC5A9C8" Ref="D?"  Part="1"
+AR Path="/5BA6E8FB/5BC5A9C8" Ref="D206"  Part="1"
+F 0 "D206" V 6446 8821 50  0000 R CNN
+F 1 "LL4148" V 6355 8821 50  0000 R CNN
+F 2 "pap:D_MiniMELF" H 6400 8725 50  0001 C CNN
+F 3 "http://www.vishay.com/docs/85557/ll4148.pdf" H 6400 8900 50  0001 C CNN
+	1    6400 8900
+	0    -1   -1   0
+$EndComp
+Wire Wire Line
+	5900 8550 5900 8750
+Wire Wire Line
+	6200 8650 6400 8650
+Wire Wire Line
+	6400 8650 6400 8750
+Connection ~ 6200 8650
+Wire Wire Line
+	6200 8650 6200 8550
+Wire Wire Line
+	6400 9050 6400 9150
+Wire Wire Line
+	6400 9150 6600 9150
+Wire Wire Line
+	6600 9150 6600 8550
 $EndSCHEMATC

Commit message: cambio de nombres, mejorop serigrafia, agrego pin
agrego el pin de flag ya que me sobraba un pin en el RJ12, cambio los
nombres de 0-50 para motor y 51 a 100 para conector, ajusto el espesor
de la seri, y algunas cosas mas..
Parts:
- added JP2: jumper, pap:SolderJumper-2_P1.3mm_Open_RoundedPad1.0x1.5mm, symbol Jumper:SolderJumper_2_Open
- renumbered D204 to D13, D202 to D14, D205 to D15, D206 to D16, D201 to D17, D203 to D9, R201 to R1
Connections:
- net labels added: Vreg
- wire segments 143 -> 149
Other:
- note added: "Asignacino de Flags \nde power"
- note added: "Leds\n"
- note added: "Power"
- note added: "Selecciono si el regulador \ninterno alimenta la logica o \nse toma desde el conector \nexterno"
- note removed: "Leds debug\n"
Changed lines of the file:
@@
 	7000 4000 7150 4000
-$Comp
-L pap:3V3 #PWR?
-U 1 1 5BA71FD4
-P 8200 3600
-AR Path="/5BA71FD4" Ref="#PWR?"  Part="1"
-AR Path="/5BA6E8FB/5BA71FD4" Ref="#PWR0129"  Part="1"
-F 0 "#PWR0129" H 8200 3500 50  0001 C CNN
-F 1 "3V3" H 8200 3875 50  0000 C CNN
-F 2 "" H 8200 3600 50  0001 C CNN
-F 3 "" H 8200 3600 50  0001 C CNN
-	1    8200 3600
-	1    0    0    -1
-$EndComp
 $Comp
 L Device:R R6
@@
 Wire Wire Line
 	1400 9250 1400 9350
-Text Label 2100 9400 3    50   ~ 0
-Flag
 Text HLabel 1000 9350 3    50   Input ~ 0
 CS
@@
 Text Notes 5450 1250 0    197  ~ 39
 Motor Driver IC
-Text Notes 2100 8000 0    197  ~ 39
-Leds debug\n
+Text Notes 2450 7900 0    197  ~ 39
+Leds\n
 Text Notes 2250 9850 0    50   ~ 0
 Contemplo leds para ver movimiento en \nsincro con el motor mas algunos de debug \ncomo flag\n
@@
 Wire Wire Line
 	7000 4100 7300 4100
-Text Label 2650 4200 2    50   ~ 0
-Flag
 Wire Wire Line
 	2650 4200 3150 4200
@@
 	8400 8650 8550 8650
 $Comp
-L Device:R R201
+L Device:R R1
 U 1 1 5BBC4586
 P 9350 9000
-F 0 "R201" V 9150 9000 50  0000 C CNN
+F 0 "R1" V 9150 9000 50  0000 C CNN
 F 1 "R" V 9250 9000 50  0000 C CNN
 F 2 "pap:R_0805_2012Metric" V 9280 9000 50  0001 C CNN
@@
 P 8250 8650
 AR Path="/5BCB0C65" Ref="D?"  Part="1"
-AR Path="/5BA6E8FB/5BCB0C65" Ref="D201"  Part="1"
-F 0 "D201" H 8250 8866 50  0000 C CNN
+AR Path="/5BA6E8FB/5BCB0C65" Ref="D17"  Part="1"
+F 0 "D17" H 8250 8866 50  0000 C CNN
 F 1 "LL4148" H 8250 8775 50  0000 C CNN
 F 2 "pap:D_MiniMELF" H 8250 8475 50  0001 C CNN
@@
 Busy
 $Comp
-L Device:LED D203
+L Device:LED D9
 U 1 1 5BB9D2E4
 P 1750 8800
-F 0 "D203" V 1788 8683 50  0000 R CNN
+F 0 "D9" V 1788 8683 50  0000 R CNN
 F 1 "LED" V 1697 8683 50  0000 R CNN
 F 2 "pap:led5p_rj" H 1750 8800 50  0001 C CNN
@@
 $EndComp
 $Comp
-L Device:LED D204
+L Device:LED D13
 U 1 1 5BBA7BC3
 P 2450 8800
-F 0 "D204" V 2488 8683 50  0000 R CNN
+F 0 "D13" V 2488 8683 50  0000 R CNN
 F 1 "LED" V 2397 8683 50  0000 R CNN
 F 2 "pap:led5p_rj" H 2450 8800 50  0001 C CNN
@@
 $EndComp
 $Comp
-L pap:LED_I D202
+L pap:LED_I D14
 U 1 1 5BC42DA3
 P 4600 8750
-F 0 "D202" V 4638 8633 50  0000 R CNN
+F 0 "D14" V 4638 8633 50  0000 R CNN
 F 1 "LED_I" V 4547 8633 50  0000 R CNN
 F 2 "pap:led5p_enchufable" H 4600 8750 50  0001 C CNN
@@
 P 5900 8900
 AR Path="/5BC459B0" Ref="D?"  Part="1"
-AR Path="/5BA6E8FB/5BC459B0" Ref="D205"  Part="1"
-F 0 "D205" V 5946 8821 50  0000 R CNN
+AR Path="/5BA6E8FB/5BC459B0" Ref="D15"  Part="1"
+F 0 "D15" V 5946 8821 50  0000 R CNN
 F 1 "LL4148" V 5855 8821 50  0000 R CNN
 F 2 "pap:D_MiniMELF" H 5900 8725 50  0001 C CNN
@@
 P 6400 8900
 AR Path="/5BC5A9C8" Ref="D?"  Part="1"
-AR Path="/5BA6E8FB/5BC5A9C8" Ref="D206"  Part="1"
-F 0 "D206" V 6446 8821 50  0000 R CNN
+AR Path="/5BA6E8FB/5BC5A9C8" Ref="D16"  Part="1"
+F 0 "D16" V 6446 8821 50  0000 R CNN
 F 1 "LL4148" V 6355 8821 50  0000 R CNN
 F 2 "pap:D_MiniMELF" H 6400 8725 50  0001 C CNN
@@
 Wire Wire Line
 	6600 9150 6600 8550
+$Comp
+L pap:Vreg #PWR0121
+U 1 1 5BCED205
+P 8200 3600
+F 0 "#PWR0121" H 8200 3900 50  0001 C CNN
+F 1 "Vreg" H 8200 3875 50  0000 C CNN
+F 2 "" H 7850 3450 50  0001 C CNN
+F 3 "" H 7850 3450 50  0001 C CNN
+	1    8200 3600
+	1    0    0    -1
+$EndComp
+Text HLabel 2650 4200 0    50   Input ~ 0
+Flag
+Text HLabel 2100 9400 3    50   Input ~ 0
+Flag
+$Comp
+L pap:Vreg #PWR?
+U 1 1 5BCFBE1E
+P 12300 8400
+AR Path="/5BA6E5CE/5BCFBE1E" Ref="#PWR?"  Part="1"
+AR Path="/5BA6E8FB/5BCFBE1E" Ref="#PWR0122"  Part="1"
+F 0 "#PWR0122" H 12300 8700 50  0001 C CNN
+F 1 "Vreg" H 12300 8675 50  0000 C CNN
+F 2 "" H 11950 8250 50  0001 C CNN
+F 3 "" H 11950 8250 50  0001 C CNN
+	1    12300 8400
+	1    0    0    -1
+$EndComp
+$Comp
+L Jumper:SolderJumper_2_Open JP?
+U 1 1 5BCFBE25
+P 12600 8500
+AR Path="/5BA6E5CE/5BCFBE25" Ref="JP?"  Part="1"
+AR Path="/5BA6E8FB/5BCFBE25" Ref="JP2"  Part="1"
+F 0 "JP2" H 12600 8275 50  0000 C CNN
+F 1 "jumper" H 12600 8366 50  0000 C CNN
+F 2 "pap:SolderJumper-2_P1.3mm_Open_RoundedPad1.0x1.5mm" H 12600 8500 50  0001 C CNN
+F 3 "~" H 12600 8500 50  0001 C CNN
+	1    12600 8500
+	-1   0    0    1
+$EndComp
+Wire Wire Line
+	12450 8500 12300 8500
+$Comp
+L pap:3V3 #PWR?
+U 1 1 5BCFBE2D
+P 12900 8400
+AR Path="/5BCFBE2D" Ref="#PWR?"  Part="1"
+AR Path="/5BA6E8FB/5BCFBE2D" Ref="#PWR0123"  Part="1"
+AR Path="/5BA6E5CE/5BCFBE2D" Ref="#PWR?"  Part="1"
+F 0 "#PWR0123" H 12900 8300 50  0001 C CNN
+F 1 "3V3" H 12900 8675 50  0000 C CNN
+F 2 "" H 12900 8400 50  0001 C CNN
+F 3 "" H 12900 8400 50  0001 C CNN
+	1    12900 8400
+	1    0    0    -1
+$EndComp
+Wire Wire Line
+	12900 8500 12750 8500
+Text Notes 13250 7850 0    197  ~ 39
+Power
+Wire Wire Line
+	12900 8500 12900 8400
+Wire Wire Line
+	12300 8400 12300 8500
+$Comp
+L pap:3V3 #PWR?
+U 1 1 5BD1F950
+P 13600 8450
+AR Path="/5BD1F950" Ref="#PWR?"  Part="1"
+AR Path="/5BA6E8FB/5BD1F950" Ref="#PWR0124"  Part="1"
+AR Path="/5BA6E5CE/5BD1F950" Ref="#PWR?"  Part="1"
+F 0 "#PWR0124" H 13600 8350 50  0001 C CNN
+F 1 "3V3" H 13600 8725 50  0000 C CNN
+F 2 "" H 13600 8450 50  0001 C CNN
+F 3 "" H 13600 8450 50  0001 C CNN
+	1    13600 8450
+	1    0    0    -1
+$EndComp
+$Comp
+L pap:G3V3 #PWR?
+U 1 1 5BD2633F
+P 14500 8300
+AR Path="/5BD2633F" Ref="#PWR?"  Part="1"
+AR Path="/5BA6E8FB/5BD2633F" Ref="#PWR0125"  Part="1"
+F 0 "#PWR0125" H 14500 8050 50  0001 C CNN
+F 1 "G3V3" H 14505 8127 50  0000 C CNN
+F 2 "" H 14500 8300 50  0001 C CNN
+F 3 "" H 14500 8300 50  0001 C CNN
+	1    14500 8300
+	1    0    0    -1
+$EndComp
+$Comp
+L power:PWR_FLAG #FLG0103
+U 1 1 5BD2DE1B
+P 13800 8350
+AR Path="/5BA6E8FB/5BD2DE1B" Ref="#FLG0103"  Part="1"
+AR Path="/5BA6E5CE/5BD2DE1B" Ref="#FLG?"  Part="1"
+F 0 "#FLG0103" H 13800 8425 50  0001 C CNN
+F 1 "PWR_FLAG" H 13868 8394 50  0000 L CNN
+F 2 "" H 13800 8350 50  0001 C CNN
+F 3 "~" H 13800 8350 50  0001 C CNN
+	1    13800 8350
+	1    0    0    -1
+$EndComp
+Wire Wire Line
+	13600 8450 13800 8450
+Wire Wire Line
+	13800 8450 13800 8350
+$Comp
+L power:PWR_FLAG #FLG0104
+U 1 1 5BD39DC3
+P 14500 8300
+AR Path="/5BA6E8FB/5BD39DC3" Ref="#FLG0104"  Part="1"
+AR Path="/5BA6E5CE/5BD39DC3" Ref="#FLG?"  Part="1"
+F 0 "#FLG0104" H 14500 8375 50  0001 C CNN
+F 1 "PWR_FLAG" H 14500 8474 50  0000 C CNN
+F 2 "" H 14500 8300 50  0001 C CNN
+F 3 "~" H 14500 8300 50  0001 C CNN
+	1    14500 8300
+	1    0    0    -1
+$EndComp
+Wire Notes Line
+	15250 7500 15250 9400
+Wire Notes Line
+	15250 9400 12000 9400
+Wire Notes Line
+	12000 9400 12000 7500
+Wire Notes Line
+	12000 7500 15250 7500
+Text Notes 12150 8950 0    50   ~ 0
+Selecciono si el regulador \ninterno alimenta la logica o \nse toma desde el conector \nexterno
+Text Notes 13600 8800 0    50   ~ 0
+Asignacino de Flags \nde power
 $EndSCHEMATC

Commit message: agrego gerbers.. va quedando peeero falta crc de layout
ahi lo voy liquidando, me convence, pero me falta tirar el crc en layout
que tiene muchos errores principalmente por el tema de que para una
misma net tengo varias restriccinoes solapadas.. vere como hago con eso
y lo cierro.. ser maniana.. me estoy durmiendo..
ha, cambio tambien un poco la jerarquia de dirs asi queda mas ordenadito
Changed lines of the file:
@@
 EESchema Schematic File Version 4
-LIBS:pap-cache
 EELAYER 26 0
 EELAYER END
@@
 L pap:G3V3 #PWR?
 U 1 1 5BD2633F
-P 14500 8300
+P 14600 8350
 AR Path="/5BD2633F" Ref="#PWR?"  Part="1"
 AR Path="/5BA6E8FB/5BD2633F" Ref="#PWR0125"  Part="1"
-F 0 "#PWR0125" H 14500 8050 50  0001 C CNN
-F 1 "G3V3" H 14505 8127 50  0000 C CNN
-F 2 "" H 14500 8300 50  0001 C CNN
-F 3 "" H 14500 8300 50  0001 C CNN
-	1    14500 8300
+F 0 "#PWR0125" H 14600 8100 50  0001 C CNN
+F 1 "G3V3" H 14605 8177 50  0000 C CNN
+F 2 "" H 14600 8350 50  0001 C CNN
+F 3 "" H 14600 8350 50  0001 C CNN
+	1    14600 8350
 	1    0    0    -1
 $EndComp
@@
 L power:PWR_FLAG #FLG0104
 U 1 1 5BD39DC3
-P 14500 8300
+P 14600 8350
 AR Path="/5BA6E8FB/5BD39DC3" Ref="#FLG0104"  Part="1"
 AR Path="/5BA6E5CE/5BD39DC3" Ref="#FLG?"  Part="1"
-F 0 "#FLG0104" H 14500 8375 50  0001 C CNN
-F 1 "PWR_FLAG" H 14500 8474 50  0000 C CNN
-F 2 "" H 14500 8300 50  0001 C CNN
-F 3 "~" H 14500 8300 50  0001 C CNN
-	1    14500 8300
-	1    0    0    -1
-$EndComp
+F 0 "#FLG0104" H 14600 8425 50  0001 C CNN
+F 1 "PWR_FLAG" H 14600 8524 50  0000 C CNN
+F 2 "" H 14600 8350 50  0001 C CNN
+F 3 "~" H 14600 8350 50  0001 C CNN
+	1    14600 8350
+	1    0    0    -1
+$EndComp

Commit message: me habia olvidado algunos capas, agrego leds, me falta aun
no estaba poniendo los descaoples de los reguladores internos y hay uno
de 220uF! ese lo mando TH, igual voy a verificar en el PCB de st. pero
igual me faltaban tambien los capas de 3v3 y 85v tambien.. veo donde los
meto
Parts:
- added C2, C7, C8, C9, C?: C, pap:C_0805_2012Metric, symbol Device:C
- added C3: 220uFx25v, Capacitor_THT:CP_Radial_D6.3mm_P2.50mm, symbol Device:C
- added D1, D18: LED_SMD, pap:Wo_Paste_LED_0805_2012Metric_Pad1.15x1.40mm_HandSolder, symbol pap:LED_I
- added R15: R, pap:R_0805_2012Metric, symbol Device:R
- added R2, R5: R, pap:Wo_Paste_R_0805_2012Metric_Pad1.15x1.40mm_HandSolder, symbol Device:R
Connections:
- wire segments 149 -> 171
Other:
- note added: "SMD internos para debug\nNo se montan en p&p ni en produccion\npara soldado manual en lab"

Commit message: termino ruteo, genero gerbers y drills, y entrego
Listo pisto, lo dejo asi, ya lo revise varias veces, agregue los
desacoples y el bulk pendiente, coloreo leds con nuevo 3d, genero
gerners, y agrego valores a los componentes. ha y tambien dejo PTH los
agujeros de los tornillos, quedan mejor. y no mucho mas.. entrego ya!
Parts:
- added C11: C, pap:C_0805_2012Metric, symbol Device:C
- C1: value C -> 10n
- C3: footprint Capacitor_THT:CP_Radial_D6.3mm_P2.50mm -> pap:CP_Radial_D6.3mm_P2.50mm
- C4, C5: value C -> 220n
- C6, C9: value C -> 100n
- D10, D7: footprint pap:led5p_enchufable -> pap:led5x2_enchufable_amarillo
- D11, D8: footprint pap:led5p_enchufable -> pap:led5x2_enchufable_verde
- D12: value D_Zener -> 3v3
- D13, D4: footprint pap:led5p_rj -> pap:led5x2_rj_verde
- D14: footprint pap:led5p_enchufable -> pap:led5x2_enchufable_rojo
- D5, D6: footprint pap:led5p_rj -> pap:led5x2_rj_amarillo
- D9: footprint pap:led5p_rj -> pap:led5x2_rj_rojo_abierto
- R1, R11, R12, R13, R14: value R -> 10k
- R10, R5, R8, R9: value R -> 100e
- R16: renamed from R203; value R -> 100e
- R17: renamed from R204; value R -> 100e
- R18: renamed from R202; value R -> 10k
- R2: value R -> 1k5
- R3, R4: value R -> 0.1e
- R6: value R -> 100k
- R7: value R -> 3k3
- gave numbers to parts that had none: 1
Connections:
- wire segments 171 -> 173
Other:
- note added: "Bulk y desacople\nen 15v"
- note added: "Bulk y desacople\nen 85v"
- note added: "Desacoples\nen 3v3"
- note added: "Es open drain, \nagrego pullup"
- note added: "Leds de debug \nrepresentativos"
- note added: "Leds en sincro con \nlos motores"
- note removed: "Contemplo leds para ver movimiento en \nsincro con el motor mas algunos de debug \ncomo flag\n"
