File: motor.sch (KiCad schematic (older format))
At the start: 49 parts, among them U1 powerstep01

Commit message: agfego valores faltantes de capas
Gracias al aporte de Gonzalo, me habian quedado algunos capas sin valor.
.Corrijo. Hay otras sugerencias de Gonzalo que no se corrigen, solo se
consideran y se evaluaran luego
Parts:
- C10, C11, C2, C7, C8: value C -> 100n
Other:
- note added: "Asignacion de Flags \nde power"
- note removed: "Asignacino de Flags \nde power"
Changed lines of the file:
@@
 Selecciono si el regulador \ninterno alimenta la logica o \nse toma desde el conector \nexterno
 Text Notes 12050 2150 0    50   ~ 0
-Asignacino de Flags \nde power
+Asignacion de Flags \nde power
 $Comp
 L Device:R R2
@@
 AR Path="/5BA6E8FB/5BC8BB43" Ref="C7"  Part="1"
 F 0 "C7" H 11935 6254 50  0000 R CNN
-F 1 "C" H 11935 6345 50  0000 R CNN
+F 1 "100n" H 11935 6345 50  0000 R CNN
 F 2 "pap:C_0805_2012Metric" H 12088 6150 50  0001 C CNN
 F 3 "~" H 12050 6300 50  0001 C CNN
@@
 AR Path="/5BA6E8FB/5BC8BE5B" Ref="C8"  Part="1"
 F 0 "C8" H 11435 6254 50  0000 R CNN
-F 1 "C" H 11435 6345 50  0000 R CNN
+F 1 "100n" H 11435 6345 50  0000 R CNN
 F 2 "pap:C_0805_2012Metric" H 11588 6150 50  0001 C CNN
 F 3 "~" H 11550 6300 50  0001 C CNN
@@
 AR Path="/5BA6E8FB/5BC8BED1" Ref="C2"  Part="1"
 F 0 "C2" H 11085 6254 50  0000 R CNN
-F 1 "C" H 11085 6345 50  0000 R CNN
+F 1 "100n" H 11085 6345 50  0000 R CNN
 F 2 "pap:C_0805_2012Metric" H 11238 6150 50  0001 C CNN
 F 3 "~" H 11200 6300 50  0001 C CNN
@@
 U 1 1 5BCD74EE
 P 13600 6300
-F 0 "R15" V 13400 6300 50  0000 C CNN
-F 1 "R" V 13500 6300 50  0000 C CNN
+F 0 "R15" H 13530 6254 50  0000 R CNN
+F 1 "R" H 13530 6345 50  0000 R CNN
 F 2 "pap:R_0805_2012Metric" V 13530 6300 50  0001 C CNN
 F 3 "~" H 13600 6300 50  0001 C CNN
@@
 AR Path="/5BA6E8FB/5BCFE386" Ref="C10"  Part="1"
 F 0 "C10" H 14085 6204 50  0000 R CNN
-F 1 "C" H 14085 6295 50  0000 R CNN
+F 1 "100n" H 14085 6295 50  0000 R CNN
 F 2 "pap:C_0805_2012Metric" H 14238 6100 50  0001 C CNN
 F 3 "~" H 14200 6250 50  0001 C CNN
@@
 AR Path="/5BA6E8FB/5BC93D4F" Ref="C11"  Part="1"
 F 0 "C11" H 14535 6204 50  0000 R CNN
-F 1 "C" H 14535 6295 50  0000 R CNN
+F 1 "100n" H 14535 6295 50  0000 R CNN
 F 2 "pap:C_0805_2012Metric" H 14688 6100 50  0001 C CNN
 F 3 "~" H 14650 6250 50  0001 C CNN
